Commit message: <feat>Add underwater dynamics feature for simulating gimbalrotor

File: robots/gimbalrotor/robots/bi/gimbalrotor.gazebo.xacro (robot description, xacro)
@@ -1,9 +1,24 @@
 <?xml version="1.0"?>
-<robot
-    xmlns:xacro="http://www.ros.org/wiki/xacro" name="gimbalrotor" >
+<robot name="gimbalrotor" xmlns:xacro="http://www.ros.org/wiki/xacro" >
   <xacro:arg name="robot_name" default="gimbalrotor" />
+  <!-- include the basic urdf -->
   <xacro:include filename="$(find gimbalrotor)/robots/bi/gimbalrotor.urdf.xacro" />
-  <!-- gazebo plugin for default controller and sensors -->
+  <!-- include hydrodynamics params -->
+  <xacro:include filename="$(find gimbalrotor)/urdf/bi/gimbalrotor_hydro.xacro" />
+  <!-- include spinal controller -->
   <xacro:include filename="$(find aerial_robot_simulation)/xacro/spinal.gazebo.xacro" />
   <xacro:gazebo_spinal robot_name="$(arg robot_name)" mag_frame="fc" />
+   <!-- underwater plugin -->
+  <xacro:gimbalrotor_default>
+    <gazebo>
+      <plugin name="uuv_plugin" filename="libuuv_underwater_object_ros_plugin.so">
+        <fluid_density>1028.0</fluid_density>
+        <flow_velocity_topic>hydrodynamics/current_velocity</flow_velocity_topic>
+        <debug>1</debug>
+        <verbose>true</verbose>
+        <!-- apply the hydronamic model -->
+        <xacro:gimbalrotor_hydro_model namespace="$(arg robot_name)" />
+      </plugin>
+    </gazebo>
+  </xacro:gimbalrotor_default>
 </robot>

File: robots/gimbalrotor/robots/bi/gimbalrotor.urdf.xacro (robot description, xacro)
@@ -1,5 +1,5 @@
 <?xml version="1.0"?>
-<robot
-    xmlns:xacro="http://www.ros.org/wiki/xacro" name="gimbalrotor" >
+<robot xmlns:xacro="http://www.ros.org/wiki/xacro">
+<xacro:macro name="gimbalrotor_default" params="*gazebo" >
   <xacro:include filename="$(find gimbalrotor)/urdf/bi/gimbalrotor.urdf.xacro" />
   <xacro:include filename="$(find gimbalrotor)/urdf/bi/common.xacro" />
@@ -7,3 +7,6 @@
   <xacro:gimbalrotor_thrust_link self="1" rotor_direction="1"/>
   <xacro:gimbalrotor_thrust_link self="2" rotor_direction="-1"/>
+  <!-- Set up hydrodynamic plugin given as input parameter -->
+  <xacro:insert_block name="gazebo"/>
+</xacro:macro>
 </robot>
