Commit message: [Gimbalrotor][bi] update the urdf of bi-copter

File: robots/gimbalrotor/urdf/bi/gimbalrotor.urdf.xacro (robot description, xacro)
@@ -17,13 +17,16 @@
     <link name="base_link">
       <inertial>
-        <origin xyz="0 0 -0.134417" rpy="0 0 0"/>
-        <mass value="0.942442"/>
-        <inertia
-            ixx="0.015351" iyy="0.002766" izz="0.013177"
-            ixy="-0.000002" ixz="-0.000024" iyz="0.000002"/>
+      <!-- origin xyz is the xyz of cog of this link -->
+      <!-- so the root of this system should be aligned with geometry center of your design? -->
+      <!-- for base_link, the origin may should be aligned with the cog? so that we can get the inertial of co -->
+        <origin xyz="0 0 -0.0369" rpy="0 0 0"/>
+        <mass value="0.859"/>
+        <inertia
+            ixx="0.014901" iyy="0.002396" izz="0.013177"
+            ixy="-0.00002" ixz="-0.00085" iyz="0.000003"/>
       </inertial>
       <visual>
         <geometry>
-          <mesh filename="package://gimbalrotor/urdf/bi/mesh/kxr_flight_unit_base_link.dae" scale="0.001 0.001 0.001"/>
+          <mesh filename="package://gimbalrotor/urdf/bi/mesh/base_link.dae"/>
           <origin xyz="0 0 0" rpy="0 0 0"/>
         </geometry>
@@ -84,5 +87,7 @@
       <parent link="base_link" />
       <child link="rotor_arm${child1}"/>
+      <!-- from base_link to rotor_arm cord -->
       <origin xyz="0 0.154 0.051" rpy="0 0 ${pi/2}"/>
+      <!-- axis的意思是此joint的可動關節的方向，也就是自由度的方向 -->
       <axis xyz="0 0 1"/>
     </joint>
@@ -99,4 +104,5 @@
       <child link="gimbal_link${child1}"/>
       <origin xyz="0 0 0" rpy="0 0 0"/>
+      <!-- after the rotation of cord, the dof right now exists in x axis -->
       <axis xyz="1 0 0"/>
       <dynamics damping="0.8" friction="0.0"/>
@@ -141,9 +147,10 @@
         <mass value="0.250950"/>
         <inertia
-            ixx="0.001920" iyy="0.000249" izz="0.013177"
-            ixy="0.000002" ixz="-0.000024" iyz="0.000002"/>
+            ixx="0.000378" iyy="0.000226" izz="0.000503"
+            ixy="0.00000" ixz="-0.00000" iyz="0.00000"/>
       </inertial>
       <visual>
         <origin xyz="0 0 0" rpy="0 0 ${-pi/2}"/>
+        <!-- existence of scale is because of the unit of export(mm or m)   -->
         <geometry>
           <mesh filename="package://gimbalrotor/urdf/bi/mesh/thrust_link_left_straight.dae" scale="0.001 0.001 0.001"/>

Commit message: [Gimbalrotor] update the urdf to fit for gazebo

File: robots/gimbalrotor/urdf/bi/gimbalrotor.urdf.xacro (robot description, xacro)
@@ -33,5 +33,5 @@
       </visual>
       <collision>
-        <origin xyz="0 0 0" rpy="0 0 0"/>
+        <origin xyz="0 0 0.0369" rpy="0 0 0"/>
         <geometry>
           <box size="0.1 0.3 0.21"/>

Commit message: [gimbalrotor] modify the urdf and config for real machine

File: robots/gimbalrotor/urdf/bi/gimbalrotor.urdf.xacro (robot description, xacro)
@@ -20,18 +20,18 @@
       <!-- so the root of this system should be aligned with geometry center of your design? -->
       <!-- for base_link, the origin may should be aligned with the cog? so that we can get the inertial of co -->
-        <origin xyz="0 0 -0.0369" rpy="0 0 0"/>
-        <mass value="0.859"/>
-        <inertia
-            ixx="0.014901" iyy="0.002396" izz="0.013177"
-            ixy="-0.00002" ixz="-0.00085" iyz="0.000003"/>
+        <origin xyz="-0.001881 -0.000360 -0.034200" rpy="0 0 0"/>
+        <mass value="0.856021"/>
+        <inertia
+            ixx="0.013681" iyy="0.002270" izz="0.013685"
+            ixy="-0.00001" ixz="-0.00074" iyz="-0.000003"/>
       </inertial>
       <visual>
         <geometry>
-          <mesh filename="package://gimbalrotor/urdf/bi/mesh/base_link.dae"/>
+          <mesh filename="package://gimbalrotor/urdf/bi/mesh/BaseLinkNew.dae"/>
           <origin xyz="0 0 0" rpy="0 0 0"/>
         </geometry>
       </visual>
       <collision>
-        <origin xyz="0 0 0.0369" rpy="0 0 0"/>
+        <origin xyz="0 0 -0.5369" rpy="0 0 0"/>
         <geometry>
           <box size="0.1 0.3 0.21"/>
@@ -80,5 +80,5 @@
       <parent link="base_link"/>
       <child link="fc"/>
-      <origin xyz="0 0 0" rpy="0 0 0"/>
+      <origin xyz="0.025 -0.02598 0.0438" rpy="0 0 0"/>
       <axis xyz="0 0 1"/>
     </joint>
@@ -89,5 +89,4 @@
       <!-- from base_link to rotor_arm cord -->
       <origin xyz="0 0.154 0.051" rpy="0 0 ${pi/2}"/>
-      <!-- axis的意思是此joint的可動關節的方向，也就是自由度的方向 -->
       <axis xyz="0 0 1"/>
     </joint>
@@ -104,5 +103,4 @@
       <child link="gimbal_link${child1}"/>
       <origin xyz="0 0 0" rpy="0 0 0"/>
-      <!-- after the rotation of cord, the dof right now exists in x axis -->
       <axis xyz="1 0 0"/>
       <dynamics damping="0.8" friction="0.0"/>

Commit message: [gimbalrotor] update the urdf of gimbalrotor

File: robots/gimbalrotor/urdf/bi/gimbalrotor.urdf.xacro (robot description, xacro)
@@ -17,9 +17,9 @@
     <link name="base_link">
       <inertial>
-        <origin xyz="0 0 -0.134417" rpy="0 0 0"/>
-        <mass value="0.942442"/>
-        <inertia
-            ixx="0.015351" iyy="0.002766" izz="0.013177"
-            ixy="-0.000002" ixz="-0.000024" iyz="0.000002"/>
+      <origin xyz="-0.001881 -0.000360 -0.034200" rpy="0 0 0"/>
+        <mass value="0.856021"/>
+        <inertia
+            ixx="0.013681" iyy="0.002270" izz="0.013685"
+            ixy="-0.00001" ixz="-0.00074" iyz="-0.000003"/>
       </inertial>
       <visual>
@@ -77,5 +77,5 @@
       <parent link="base_link"/>
       <child link="fc"/>
-      <origin xyz="0 0 0" rpy="0 0 0"/>
+      <origin xyz="0.025 -0.02598 0.0438" rpy="0 0 0"/>
       <axis xyz="0 0 1"/>
     </joint>
