Commit message: [flamingo] temporarily only include the underwater motor as No. 1&2 thrst  for quick tuning and modify indeices of  pwm port for aquatic rotor to targte_pwm_[0] and  targte_pwm_[1] in attitude controller

File: robots/flamingo/urdf/flamingo.urdf copy.xacro (robot description, xacro)
@@ -181,5 +181,5 @@
     <xacro:damping_factor link="thrust${self}"/>
     #### thrust link (virtual) for aquatic motor####
-  <!-- aquatic motor
+  <!-- aquatic motor-->
     <link name="thrust${self + 2}">
       <inertial>
@@ -191,5 +191,5 @@
       </inertial>
     </link>
-    <xacro:damping_factor link="thrust${self + 2}"/> -->
+    <xacro:damping_factor link="thrust${self + 2}"/>
     ## joints ##
     #### rotor parent link joint (virtual) ####
@@ -202,19 +202,18 @@
     #### rotor joint (virtual) for aerial rotor ####
     <joint name="rotor${self}" type="continuous">
+      <limit effort="100.0" lower="${air_min_force}" upper="${air_max_force}" velocity="0.5"/>
+      <parent link="rotor_parent${self}"/>
+      <child link="thrust${self}"/>
+      <origin rpy="0 0 0" xyz="0 0 0"/>
+      <axis xyz="0 0 ${rotor_direction}"/>
+    </joint>
+    #### rotor joint (virtual) for aquatic rotor####
+    <joint name="rotor${self + 2}" type="continuous">
       <limit effort="100.0" lower="${water_min_force}" upper="${water_max_force}" velocity="0.5"/>
       <parent link="rotor_parent${self}"/>
-      <child link="thrust${self}"/>
+      <child link="thrust${self + 2}"/>
       <origin rpy="0 0 0" xyz="0 0 -0.05"/>
       <axis xyz="0 0 ${rotor_direction}"/>
     </joint>
-    #### rotor joint (virtual) for aquatic rotor####
-    <!-- <joint name="rotor${self + 2}" type="continuous"> -->
-      <!-- <limit effort="100.0" lower="${water_min_force}" upper="${water_max_force}" velocity="0.5"/> -->
-      <!-- <parent link="rotor_parent${self}"/> -->
-      <!-- <child link="thrust${self + 2}"/> -->
-      <!-- modify this position -->
-      <!-- <origin rpy="0 0 0" xyz="0 0 -0.05"/> -->
-      <!-- <axis xyz="0 0 ${rotor_direction}"/> -->
-    <!-- </joint> -->
     #### hardware interface ####
     <transmission name="rotor_tran${self}">
@@ -228,5 +227,5 @@
       </actuator>
     </transmission>
-       <!-- #### hardware interface ####
+       <!-- #### hardware interface #### -->
     <transmission name="rotor_tran${self + 2}">
       <type>transmission_interface/SimpleTransmission</type>
@@ -238,5 +237,5 @@
         <mechanicalReduction>1</mechanicalReduction>
       </actuator>
-    </transmission> -->
+    </transmission>
   </xacro:macro>
 </robot>
