Commit message: [flamingo] update the aquatic motor info for flamingo and add zero pint offset for pwm servo

File: robots/flamingo/urdf/common.xacro (robot description, xacro)
@@ -7,11 +7,11 @@
   <!-- the rotor -->
   <thrust_link name="thrust" />
-  <m_f_rate value="-0.0172" /> <!-- drug torque rate -->
+  <m_f_rate value="0.0136" /> <!-- drug torque rate -->
   <!-- aerial motor -->
   <xacro:property name="air_max_force" value="18.0" /> <!-- [N] -->
   <xacro:property name="air_min_force" value="1.0" /> <!-- [N] -->
   <!-- aquatic motor -->
-  <xacro:property name="water_max_force" value="18.0" /> <!-- [N] -->
-  <xacro:property name="water_min_force" value="1.0" /> <!-- [N] -->
+  <xacro:property name="water_max_force" value="21.1743" /> <!-- [N] -->
+  <xacro:property name="water_min_force" value="0.0" /> <!-- [N] -->
   <!-- friction -->
   <xacro:macro name="friction" params="self">

Commit message: [flamingo][controlParam] first take off param

File: robots/flamingo/urdf/common.xacro (robot description, xacro)
@@ -13,5 +13,5 @@
   <!-- aquatic motor -->
   <xacro:property name="water_max_force" value="18.0" /> <!-- [N] -->
-  <xacro:property name="water_min_force" va0.0188lue="1.0" /> <!-- [N] -->
+  <xacro:property name="water_min_force" value="1.0" /> <!-- [N] -->
   <!-- friction -->
   <xacro:macro name="friction" params="self">

Commit message: [flamingo][urdf] update inertial properties and joint origins for base and gimbal links

File: robots/flamingo/urdf/common.xacro (robot description, xacro)
@@ -7,11 +7,11 @@
   <!-- the rotor -->
   <thrust_link name="thrust" />
-  <m_f_rate value="-0.0172" /> <!-- drug torque rate -->
+  <m_f_rate value="0.0188" /> <!-- drug torque rate -->
   <!-- aerial motor -->
-  <xacro:property name="air_max_force" value="18.0" /> <!-- [N] -->
+  <xacro:property name="air_max_force" value="31.72" /> <!-- [N] -->
   <xacro:property name="air_min_force" value="1.0" /> <!-- [N] -->
   <!-- aquatic motor -->
   <xacro:property name="water_max_force" value="18.0" /> <!-- [N] -->
-  <xacro:property name="water_min_force" value="1.0" /> <!-- [N] -->
+  <xacro:property name="water_min_force" va0.0188lue="1.0" /> <!-- [N] -->
   <!-- friction -->
   <xacro:macro name="friction" params="self">

File: robots/flamingo/urdf/flamingo.urdf.xacro (robot description, xacro)
@@ -18,9 +18,9 @@
       <inertial>
       <!-- define the pos of cog under the root frame -->
-        <origin xyz="-0.0597843 -0.0009927 -0.0963443" rpy="0 0 0"/>
-        <mass value="2.80011285"/>
-        <inertia
-            ixx="0.0139299" iyy="0.0514116" izz="0.0436979"
-            ixy="0.0000038" ixz="0.0001678" iyz="-0.0000065"/>
+        <origin xyz="-0.1320295 0.0020275 -0.1049664" rpy="0 0 0"/>
+        <mass value="2.7914918"/>
+        <inertia
+            ixx="0.0151463" iyy="0.0558584" izz="0.0469160"
+            ixy="0.0000036" ixz="-0.0002407" iyz="0.0000023"/>
       </inertial>
       <visual>
@@ -31,7 +31,7 @@
       </visual>
       <collision>
-        <origin xyz="-0.07191 0.0069 -0.08959" rpy="0 0 0"/>
-        <geometry>
-          <box size="0.4641 0.158 0.31219"/>
+        <origin xyz="-0.13009 0.0059 -0.08959" rpy="0 0 0"/>
+        <geometry>
+          <box size="0.4671 0.168 0.33266"/>
         </geometry>
       </collision>
@@ -77,5 +77,5 @@
       <parent link="base_link"/>
       <child link="fc"/>
-      <origin xyz="-0.07191 0.0069 -0.08959" rpy="0 0 ${-0.5 * pi}"/>
+      <origin xyz="-0.101 0.023 -0.09983" rpy="0 0 ${-0.5 * pi}"/>
       <axis xyz="0 0 1"/>
     </joint>
@@ -85,5 +85,5 @@
       <parent link="base_link" />
       <child link="rotor_arm${child1}"/>
-      <origin xyz="0.16605 -0.0011 0.045" rpy="0 0 0"/>
+      <origin xyz="0.09665 0.0021 0.045" rpy="0 0 0"/>
       <axis xyz="0 0 1"/>
     </joint>
@@ -91,5 +91,5 @@
       <parent link="base_link"/>
       <child link="rotor_arm${child2}"/>
-      <origin xyz="-0.29805 -0.0011 0.045" rpy="0 0 ${pi}"/>
+      <origin xyz="-0.36955 -0.0021 0.045" rpy="0 0 ${pi}"/>
       <axis xyz="0 0 1"/>
     </joint>
@@ -140,9 +140,9 @@
     <!-- this link's cordinate is the actual gimbal -->
       <inertial>
-        <origin xyz="0.0328427 -0.0000782 -0.0167858" rpy="0 0 0"/>
-        <mass value="0.27076"/>
-        <inertia
-            ixx="0.0007257" iyy="0.0007451" izz="0.0000987"
-            ixy="0.0000007" ixz="-0.0000189" iyz="-0.0000001"/>
+        <origin xyz="0.04005 -0.00004 -0.01307" rpy="0 0 0"/>
+        <mass value="0.29576"/>
+        <inertia
+            ixx="0.00095359" iyy="0.00099897" izz="0.00045662"
+            ixy="-0.00000035" ixz="0.00008225" iyz="-0.00000564"/>
       </inertial>
       <visual>
@@ -198,5 +198,5 @@
       <parent link="gimbal_link${self}"/>
       <child link="rotor_parent${self}"/>
-      <origin xyz="0.036 0 0" rpy="0 0 0"/>
+      <origin xyz="0.0369 0 0" rpy="0 0 0"/>
       <axis xyz="0 0 1"/>
     </joint>

Commit message: [flamingo][fix] correct thrust direction and mass influence in control calculations; update m_f_rate values in configuration files

File: robots/flamingo/urdf/common.xacro (robot description, xacro)
@@ -7,5 +7,5 @@
   <!-- the rotor -->
   <thrust_link name="thrust" />
-  <m_f_rate value="0.0136" /> <!-- drug torque rate -->
+  <m_f_rate value="-0.0136" /> <!-- drug torque rate -->
   <!-- aerial motor -->
   <xacro:property name="air_max_force" value="18.0" /> <!-- [N] -->

File: robots/flamingo/urdf/flamingo.urdf.xacro (robot description, xacro)
@@ -85,5 +85,5 @@
       <parent link="base_link"/>
       <child link="fc"/>
-      <origin xyz="-0.1181 0.01791 -0.09983" rpy="0 0 ${-0.5 * pi}"/>
+      <origin xyz="-0.1181 0.01791 -0.09983" rpy="${pi} 0 ${-0.5 * pi}"/>
       <axis xyz="0 0 1"/>
     </joint>
