Commit message: [flamingo] modify the urdf for describing the aquatic rotor

File: robots/flamingo/urdf/flamingo.urdf.xacro (robot description, xacro)
@@ -216,5 +216,5 @@
       <child link="thrust${self + 2}"/>
       <!-- modify this position -->
-      <origin rpy="0 0 0" xyz="0 0 -0.05"/>
+      <origin rpy="0 0 0" xyz="0 0 -0.02"/>
       <axis xyz="0 0 ${rotor_direction}"/>
     </joint>

Commit message: [Servo] modify the servo yaml file to avoid failed servo bridge

File: robots/flamingo/urdf/flamingo.urdf.xacro (robot description, xacro)
@@ -17,16 +17,14 @@
     <link name="base_link">
       <inertial>
-      <!-- the relative pos of cog compared to the origin of this link  -->
-      <!-- because right now the origin of base_link has been configured to  the base_link of solidworks-->
-        <origin xyz="-0.0612563 -0.0010330 -0.1010610" rpy="0 0 0"/>
-        <mass value="2.76613"/>
-        <inertia
-            ixx="0.0132295" iyy="0.0505483" izz="0.042343"
-            ixy="-0.0000062" ixz="0.0001472" iyz="0.0000005"/>
+        <origin xyz="-0.0609995 -0.0010416 -0.1022045" rpy="0 0 0"/>
+        <mass value="2.9380827"/>
+        <inertia
+            ixx="0.0134198" iyy="0.0930810" izz="0.0542620"
+            ixy=" 0.0001751" ixz="0.0184499" iyz="0.0003133"/>
       </inertial>
       <visual>
         <geometry>
           <mesh filename="package://flamingo/urdf/mesh/base_link.dae" scale="1 1 1"/>
-          <origin xyz="0.0 -0.00 0.0" rpy="0 0 0"/>
+          <origin xyz="0.0 0.0 0.0" rpy="0 0 0"/>
         </geometry>
       </visual>
@@ -183,5 +181,5 @@
     <xacro:damping_factor link="thrust${self}"/>
     #### thrust link (virtual) for aquatic motor####
-  <!-- aquatic motor -->
+  <!-- aquatic motor
     <link name="thrust${self + 2}">
       <inertial>
@@ -193,5 +191,5 @@
       </inertial>
     </link>
-    <xacro:damping_factor link="thrust${self + 2}"/>
+    <xacro:damping_factor link="thrust${self + 2}"/> -->
     ## joints ##
     #### rotor parent link joint (virtual) ####
@@ -211,12 +209,12 @@
     </joint>
     #### rotor joint (virtual) for aquatic rotor####
-    <joint name="rotor${self + 2}" type="continuous">
-      <limit effort="100.0" lower="${water_min_force}" upper="${water_max_force}" velocity="0.5"/>
-      <parent link="rotor_parent${self}"/>
-      <child link="thrust${self + 2}"/>
+    <!-- <joint name="rotor${self + 2}" type="continuous"> -->
+      <!-- <limit effort="100.0" lower="${water_min_force}" upper="${water_max_force}" velocity="0.5"/> -->
+      <!-- <parent link="rotor_parent${self}"/> -->
+      <!-- <child link="thrust${self + 2}"/> -->
       <!-- modify this position -->
-      <origin rpy="0 0 0" xyz="0 0 -0.05"/>
-      <axis xyz="0 0 ${rotor_direction}"/>
-    </joint>
+      <!-- <origin rpy="0 0 0" xyz="0 0 -0.05"/> -->
+      <!-- <axis xyz="0 0 ${rotor_direction}"/> -->
+    <!-- </joint> -->
     #### hardware interface ####
     <transmission name="rotor_tran${self}">
@@ -230,5 +228,5 @@
       </actuator>
     </transmission>
-       #### hardware interface ####
+       <!-- #### hardware interface ####
     <transmission name="rotor_tran${self + 2}">
       <type>transmission_interface/SimpleTransmission</type>
@@ -240,5 +238,5 @@
         <mechanicalReduction>1</mechanicalReduction>
       </actuator>
-    </transmission>
+    </transmission> -->
   </xacro:macro>
 </robot>

Commit message: [flamingo][urdf] update the urdf to enable upside down the fc to faciliate underwater roll target angle set

File: robots/flamingo/urdf/flamingo.urdf.xacro (robot description, xacro)
@@ -76,5 +76,5 @@
       <parent link="base_link"/>
       <child link="fc"/>
-      <origin xyz="-0.07191 0.0069 -0.08959" rpy="0 0 0"/>
+      <origin xyz="-0.07191 0.0069 -0.08959" rpy="${pi} 0 0"/>
       <axis xyz="0 0 1"/>
     </joint>

Commit message: [flamingo][urdf]update fc_joint origin to include yaw rotation for improved alignment

File: robots/flamingo/urdf/flamingo.urdf.xacro (robot description, xacro)
@@ -76,5 +76,5 @@
       <parent link="base_link"/>
       <child link="fc"/>
-      <origin xyz="-0.07191 0.0069 -0.08959" rpy="${pi} 0 0"/>
+      <origin xyz="-0.07191 0.0069 -0.08959" rpy="${pi} 0 ${0.5 * pi}"/>
       <axis xyz="0 0 1"/>
     </joint>

Commit message: [flamingo][control] invert depth control output and adjust depth error calculation for correct deth control implementation [flamingo][urdf] correct yaw rotation in fc_joint origin for accurate alignment

File: robots/flamingo/urdf/flamingo.urdf.xacro (robot description, xacro)
@@ -76,5 +76,5 @@
       <parent link="base_link"/>
       <child link="fc"/>
-      <origin xyz="-0.07191 0.0069 -0.08959" rpy="${pi} 0 ${0.5 * pi}"/>
+      <origin xyz="-0.07191 0.0069 -0.08959" rpy="${pi} 0 ${-0.5 * pi}"/>
       <axis xyz="0 0 1"/>
     </joint>

Commit message: [flamingo][urdf][controller] add desire coordinate publisher for underwater motion and update fc_joint origin for correct alignment

File: robots/flamingo/urdf/flamingo.urdf.xacro (robot description, xacro)
@@ -76,5 +76,5 @@
       <parent link="base_link"/>
       <child link="fc"/>
-      <origin xyz="-0.07191 0.0069 -0.08959" rpy="${pi} 0 ${-0.5 * pi}"/>
+      <origin xyz="-0.07191 0.0069 -0.08959" rpy="0 0 ${-0.5 * pi}"/>
       <axis xyz="0 0 1"/>
     </joint>

Commit message: [flamingo] update servo zero point offset, adjust desired roll angle for underwater motion, and modify joint origin in URDF

File: robots/flamingo/urdf/flamingo.urdf.xacro (robot description, xacro)
@@ -205,5 +205,5 @@
       <parent link="rotor_parent${self}"/>
       <child link="thrust${self}"/>
-      <origin rpy="0 0 0" xyz="0 0 -0.05"/>
+      <origin rpy="${pi} 0 0" xyz="0 0 -0.05"/>
       <axis xyz="0 0 ${rotor_direction}"/>
     </joint>

Commit message: [flamingo][refactor] update depth control parameters and joystick mappings for improved performance

File: robots/flamingo/urdf/flamingo.urdf.xacro (robot description, xacro)
@@ -205,5 +205,5 @@
       <parent link="rotor_parent${self}"/>
       <child link="thrust${self}"/>
-      <origin rpy="${pi} 0 0" xyz="0 0 -0.05"/>
+      <origin rpy="0 0 0" xyz="0 0 -0.05"/>
       <axis xyz="0 0 ${rotor_direction}"/>
     </joint>

Commit message: [flamingo][urdf] update fc_joint orientation to include rotation around Z-axis

File: robots/flamingo/urdf/flamingo.urdf.xacro (robot description, xacro)
@@ -76,5 +76,5 @@
       <parent link="base_link"/>
       <child link="fc"/>
-      <origin xyz="-0.07191 0.0069 -0.08959" rpy="0 0 0"/>
+      <origin xyz="-0.07191 0.0069 -0.08959" rpy="0 0 ${-0.5 * pi}"/>
       <axis xyz="0 0 1"/>
     </joint>

Commit message: [flamingo][urdf] update base_link inertial properties and center of gravity position

File: robots/flamingo/urdf/flamingo.urdf.xacro (robot description, xacro)
@@ -17,9 +17,10 @@
     <link name="base_link">
       <inertial>
-        <origin xyz="-0.0609995 -0.0010416 -0.1022045" rpy="0 0 0"/>
-        <mass value="2.9380827"/>
-        <inertia
-            ixx="0.0134198" iyy="0.0930810" izz="0.0542620"
-            ixy=" 0.0001751" ixz="0.0184499" iyz="0.0003133"/>
+      <!-- define the pos of cog under the root frame -->
+        <origin xyz="-0.0597843 -0.0009927 -0.0963443" rpy="0 0 0"/>
+        <mass value="2.80011285"/>
+        <inertia
+            ixx="0.0139299" iyy="0.0514116" izz="0.0436979"
+            ixy="0.0000038" ixz="0.0001678" iyz="-0.0000065"/>
       </inertial>
       <visual>

Commit message: [flamingo][urdf] update mesh filenames for base_link and thrust_unit to version 2

File: robots/flamingo/urdf/flamingo.urdf.xacro (robot description, xacro)
@@ -26,5 +26,5 @@
       <visual>
         <geometry>
-          <mesh filename="package://flamingo/urdf/mesh/base_link.dae" scale="1 1 1"/>
+          <mesh filename="package://flamingo/urdf/mesh/base_link_v2.dae" scale="1 1 1"/>
           <origin xyz="0.0 0.0 0.0" rpy="0 0 0"/>
         </geometry>
@@ -147,7 +147,7 @@
       </inertial>
       <visual>
-        <origin xyz="0.036 0.0 0.064" rpy="0 0 ${-pi/2}"/>
-        <geometry>
-          <mesh filename="package://flamingo/urdf/mesh/thrust_unit_forward.dae"/>
+        <origin xyz="0.036 0.0 0.064" rpy="0 0 0"/>
+        <geometry>
+          <mesh filename="package://flamingo/urdf/mesh/thrust_unit_v2.dae"/>
         </geometry>
       </visual>

Commit message: [flamingo][refactor] delete the bringup and urdf to be compatible with aerial mode and update the urdf for new configuration

File: robots/flamingo/urdf/flamingo.urdf.xacro (robot description, xacro)
@@ -17,20 +17,21 @@
     <link name="base_link">
       <inertial>
-        <origin xyz="-0.0609995 -0.0010416 -0.1022045" rpy="0 0 0"/>
-        <mass value="2.9380827"/>
-        <inertia
-            ixx="0.0134198" iyy="0.0930810" izz="0.0542620"
-            ixy=" 0.0001751" ixz="0.0184499" iyz="0.0003133"/>
+      <!-- define the pos of cog under the root frame -->
+        <origin xyz="-0.1320295 0.0020275 -0.1049664" rpy="0 0 0"/>
+        <mass value="2.7914918"/>
+        <inertia
+            ixx="0.0151463" iyy="0.0558584" izz="0.0469160"
+            ixy="0.0000036" ixz="-0.0002407" iyz="0.0000023"/>
       </inertial>
       <visual>
         <geometry>
-          <mesh filename="package://flamingo/urdf/mesh/base_link.dae" scale="1 1 1"/>
+          <mesh filename="package://flamingo/urdf/mesh/base_link_v2.dae" scale="1 1 1"/>
           <origin xyz="0.0 0.0 0.0" rpy="0 0 0"/>
         </geometry>
       </visual>
       <collision>
-        <origin xyz="-0.07191 0.0069 -0.08959" rpy="0 0 0"/>
-        <geometry>
-          <box size="0.4641 0.158 0.31219"/>
+        <origin xyz="-0.13009 0.0059 -0.08959" rpy="0 0 0"/>
+        <geometry>
+          <box size="0.4671 0.168 0.33266"/>
         </geometry>
       </collision>
@@ -76,5 +77,5 @@
       <parent link="base_link"/>
       <child link="fc"/>
-      <origin xyz="-0.07191 0.0069 -0.08959" rpy="0 0 ${-0.5 * pi}"/>
+      <origin xyz="-0.101 0.023 -0.09983" rpy="0 0 ${-0.5 * pi}"/>
       <axis xyz="0 0 1"/>
     </joint>
@@ -84,5 +85,5 @@
       <parent link="base_link" />
       <child link="rotor_arm${child1}"/>
-      <origin xyz="0.16605 -0.0011 0.045" rpy="0 0 0"/>
+      <origin xyz="0.09665 0.0021 0.045" rpy="0 0 0"/>
       <axis xyz="0 0 1"/>
     </joint>
@@ -90,5 +91,5 @@
       <parent link="base_link"/>
       <child link="rotor_arm${child2}"/>
-      <origin xyz="-0.29805 -0.0011 0.045" rpy="0 0 ${pi}"/>
+      <origin xyz="-0.36955 -0.0021 0.045" rpy="0 0 ${pi}"/>
       <axis xyz="0 0 1"/>
     </joint>
@@ -139,14 +140,14 @@
     <!-- this link's cordinate is the actual gimbal -->
       <inertial>
-        <origin xyz="0.0328427 -0.0000782 -0.0167858" rpy="0 0 0"/>
-        <mass value="0.27076"/>
-        <inertia
-            ixx="0.0007257" iyy="0.0007451" izz="0.0000987"
-            ixy="0.0000007" ixz="-0.0000189" iyz="-0.0000001"/>
+        <origin xyz="0.04005 -0.00004 -0.01307" rpy="0 0 0"/>
+        <mass value="0.29576"/>
+        <inertia
+            ixx="0.00095359" iyy="0.00099897" izz="0.00045662"
+            ixy="-0.00000035" ixz="0.00008225" iyz="-0.00000564"/>
       </inertial>
       <visual>
-        <origin xyz="0.036 0.0 0.064" rpy="0 0 ${-pi/2}"/>
-        <geometry>
-          <mesh filename="package://flamingo/urdf/mesh/thrust_unit_forward.dae"/>
+        <origin xyz="0.036 0.0 0.064" rpy="0 0 0"/>
+        <geometry>
+          <mesh filename="package://flamingo/urdf/mesh/thrust_unit_v2.dae"/>
         </geometry>
       </visual>
@@ -197,5 +198,5 @@
       <parent link="gimbal_link${self}"/>
       <child link="rotor_parent${self}"/>
-      <origin xyz="0.036 0 0" rpy="0 0 0"/>
+      <origin xyz="0.0369 0 0" rpy="0 0 0"/>
       <axis xyz="0 0 1"/>
     </joint>
@@ -205,5 +206,5 @@
       <parent link="rotor_parent${self}"/>
       <child link="thrust${self}"/>
-      <origin rpy="0 0 0" xyz="0 0 -0.05"/>
+      <origin rpy="0 0 0" xyz="0 0 0"/>
       <axis xyz="0 0 ${rotor_direction}"/>
     </joint>

Commit message: third take off with one battery

File: robots/flamingo/urdf/flamingo.urdf.xacro (robot description, xacro)
@@ -18,9 +18,9 @@
       <inertial>
       <!-- define the pos of cog under the root frame -->
-        <origin xyz="-0.1320295 0.0020275 -0.1049664" rpy="0 0 0"/>
-        <mass value="2.7914918"/>
-        <inertia
-            ixx="0.0151463" iyy="0.0558584" izz="0.0469160"
-            ixy="0.0000036" ixz="-0.0002407" iyz="0.0000023"/>
+        <origin xyz="-0.1325765 0.0020237 -0.1113353" rpy="0 0 0"/>
+        <mass value="3.1799818"/>
+        <inertia
+            ixx="0.0160903" iyy="0.0573578" izz="0.0476113"
+            ixy="0.0000037" ixz="-0.0001701" iyz="0.0000028"/>
       </inertial>
       <visual>

Commit message: [flamingo][urdf] update the urdf for correct fc position

File: robots/flamingo/urdf/flamingo.urdf.xacro (robot description, xacro)
@@ -77,5 +77,5 @@
       <parent link="base_link"/>
       <child link="fc"/>
-      <origin xyz="-0.101 0.023 -0.09983" rpy="0 0 ${-0.5 * pi}"/>
+      <origin xyz="-0.151 0.023 -0.09983" rpy="0 0 ${-0.5 * pi}"/>
       <axis xyz="0 0 1"/>
     </joint>

Commit message: [flamingo][controlParam] adjust control limits for xy axis and update rotor joint position in URDF

File: robots/flamingo/urdf/flamingo.urdf.xacro (robot description, xacro)
@@ -85,5 +85,5 @@
       <parent link="base_link" />
       <child link="rotor_arm${child1}"/>
-      <origin xyz="0.09665 0.0021 0.045" rpy="0 0 0"/>
+      <origin xyz="0.09665 -0.0021 0.045" rpy="0 0 0"/>
       <axis xyz="0 0 1"/>
     </joint>

Commit message: Fix joint origin coordinates for rotor coordination in URDF

File: robots/flamingo/urdf/flamingo.urdf.xacro (robot description, xacro)
@@ -85,5 +85,5 @@
       <parent link="base_link" />
       <child link="rotor_arm${child1}"/>
-      <origin xyz="0.09665 -0.0021 0.045" rpy="0 0 0"/>
+      <origin xyz="0.09665 0.0021 0.045" rpy="0 0 0"/>
       <axis xyz="0 0 1"/>
     </joint>
@@ -91,5 +91,5 @@
       <parent link="base_link"/>
       <child link="rotor_arm${child2}"/>
-      <origin xyz="-0.36955 -0.0021 0.045" rpy="0 0 ${pi}"/>
+      <origin xyz="-0.36955 0.0021 0.045" rpy="0 0 ${pi}"/>
       <axis xyz="0 0 1"/>
     </joint>

Commit message: [flamingo][urdf] adjust joint origins for fc and rotor coordination in URDF

File: robots/flamingo/urdf/flamingo.urdf.xacro (robot description, xacro)
@@ -77,5 +77,5 @@
       <parent link="base_link"/>
       <child link="fc"/>
-      <origin xyz="-0.151 0.023 -0.09983" rpy="0 0 ${-0.5 * pi}"/>
+      <origin xyz="-0.1181 0.01791 -0.09983" rpy="0 0 ${-0.5 * pi}"/>
       <axis xyz="0 0 1"/>
     </joint>
@@ -85,5 +85,5 @@
       <parent link="base_link" />
       <child link="rotor_arm${child1}"/>
-      <origin xyz="0.09665 -0.0021 0.045" rpy="0 0 0"/>
+      <origin xyz="0.09665 0.0021 0.045" rpy="0 0 0"/>
       <axis xyz="0 0 1"/>
     </joint>
@@ -91,5 +91,5 @@
       <parent link="base_link"/>
       <child link="rotor_arm${child2}"/>
-      <origin xyz="-0.36955 -0.0021 0.045" rpy="0 0 ${pi}"/>
+      <origin xyz="-0.36865 0.0021 0.045" rpy="0 0 ${pi}"/>
       <axis xyz="0 0 1"/>
     </joint>
@@ -215,5 +215,5 @@
       <!-- <child link="thrust${self + 2}"/> -->
       <!-- modify this position -->
-      <!-- <origin rpy="0 0 0" xyz="0 0 -0.05"/> -->
+      <!-- <origin rpy="0 0 0" xyz="0 0 -0.02"/> -->
       <!-- <axis xyz="0 0 ${rotor_direction}"/> -->
     <!-- </joint> -->

Commit message: [flamingo][urdf] adjust joint origins for fc and rotor coordination in URDF

File: robots/flamingo/urdf/flamingo.urdf.xacro (robot description, xacro)
@@ -77,5 +77,5 @@
       <parent link="base_link"/>
       <child link="fc"/>
-      <origin xyz="-0.151 0.023 -0.09983" rpy="0 0 ${-0.5 * pi}"/>
+      <origin xyz="-0.1181 0.01791 -0.09983" rpy="0 0 ${-0.5 * pi}"/>
       <axis xyz="0 0 1"/>
     </joint>
@@ -91,5 +91,5 @@
       <parent link="base_link"/>
       <child link="rotor_arm${child2}"/>
-      <origin xyz="-0.36955 0.0021 0.045" rpy="0 0 ${pi}"/>
+      <origin xyz="-0.36865 0.0021 0.045" rpy="0 0 ${pi}"/>
       <axis xyz="0 0 1"/>
     </joint>
@@ -215,5 +215,5 @@
       <!-- <child link="thrust${self + 2}"/> -->
       <!-- modify this position -->
-      <!-- <origin rpy="0 0 0" xyz="0 0 -0.05"/> -->
+      <!-- <origin rpy="0 0 0" xyz="0 0 -0.02"/> -->
       <!-- <axis xyz="0 0 ${rotor_direction}"/> -->
     <!-- </joint> -->

Commit message: [flamingo][urdf]Add two battery parameters in base link inertial definition for future usage

File: robots/flamingo/urdf/flamingo.urdf.xacro (robot description, xacro)
@@ -24,4 +24,12 @@
             ixy="0.0000037" ixz="-0.0001701" iyz="0.0000028"/>
       </inertial>
+        <!-- two batteries
+        <origin xyz="-0.1317508 0.0020567 -0.1162396" rpy="0 0 0"/>
+        <mass value="3.7625799"/>
+        <inertia
+            ixx="0.0176913" iyy="0.0646863" izz="0.0552197"
+            ixy="0.0000030" ixz="-0.0002878" iyz="0.0000036"/>
+      </inertial>
+ -->
       <visual>
         <geometry>

Commit message: [flamingo][cross_domain] Fix the bugs for compatible with two kinds of rotors

File: robots/flamingo/urdf/flamingo.urdf.xacro (robot description, xacro)
@@ -190,5 +190,4 @@
     <xacro:damping_factor link="thrust${self}"/>
     #### thrust link (virtual) for aquatic motor####
-  <!-- aquatic motor
     <link name="thrust${self + 2}">
       <inertial>
@@ -200,5 +199,5 @@
       </inertial>
     </link>
-    <xacro:damping_factor link="thrust${self + 2}"/> -->
+    <xacro:damping_factor link="thrust${self + 2}"/>
     ## joints ##
     #### rotor parent link joint (virtual) ####
@@ -218,12 +217,11 @@
     </joint>
     #### rotor joint (virtual) for aquatic rotor####
-    <!-- <joint name="rotor${self + 2}" type="continuous"> -->
-      <!-- <limit effort="100.0" lower="${water_min_force}" upper="${water_max_force}" velocity="0.5"/> -->
-      <!-- <parent link="rotor_parent${self}"/> -->
-      <!-- <child link="thrust${self + 2}"/> -->
-      <!-- modify this position -->
-      <!-- <origin rpy="0 0 0" xyz="0 0 -0.02"/> -->
-      <!-- <axis xyz="0 0 ${rotor_direction}"/> -->
-    <!-- </joint> -->
+    <joint name="rotor${self + 2}" type="continuous">
+      <limit effort="100.0" lower="${water_min_force}" upper="${water_max_force}" velocity="0.5"/>
+      <parent link="rotor_parent${self}"/>
+      <child link="thrust${self + 2}"/>
+      <origin rpy="0 0 0" xyz="0 0 -0.02"/>
+      <axis xyz="0 0 ${rotor_direction}"/>
+    </joint>
     #### hardware interface ####
     <transmission name="rotor_tran${self}">
@@ -237,5 +235,5 @@
       </actuator>
     </transmission>
-       <!-- #### hardware interface ####
+    #### hardware interface ####
     <transmission name="rotor_tran${self + 2}">
       <type>transmission_interface/SimpleTransmission</type>
@@ -247,5 +245,5 @@
         <mechanicalReduction>1</mechanicalReduction>
       </actuator>
-    </transmission> -->
+    </transmission>
   </xacro:macro>
 </robot>

Commit message: [flamingo][refactor] remove unused water configuration files and update FlamingoController for joystick stop command handling

File: robots/flamingo/urdf/flamingo.urdf.xacro (robot description, xacro)
@@ -18,10 +18,18 @@
       <inertial>
       <!-- define the pos of cog under the root frame -->
-        <origin xyz="-0.1320295 0.0020275 -0.1049664" rpy="0 0 0"/>
-        <mass value="2.7914918"/>
-        <inertia
-            ixx="0.0151463" iyy="0.0558584" izz="0.0469160"
-            ixy="0.0000036" ixz="-0.0002407" iyz="0.0000023"/>
-      </inertial>
+        <origin xyz="-0.1325765 0.0020237 -0.1113353" rpy="0 0 0"/>
+        <mass value="3.1799818"/>
+        <inertia
+            ixx="0.0160903" iyy="0.0573578" izz="0.0476113"
+            ixy="0.0000037" ixz="-0.0001701" iyz="0.0000028"/>
+      </inertial>
+        <!-- two batteries
+        <origin xyz="-0.1317508 0.0020567 -0.1162396" rpy="0 0 0"/>
+        <mass value="3.7625799"/>
+        <inertia
+            ixx="0.0176913" iyy="0.0646863" izz="0.0552197"
+            ixy="0.0000030" ixz="-0.0002878" iyz="0.0000036"/>
+      </inertial>
+ -->
       <visual>
         <geometry>
@@ -77,5 +85,5 @@
       <parent link="base_link"/>
       <child link="fc"/>
-      <origin xyz="-0.101 0.023 -0.09983" rpy="0 0 ${-0.5 * pi}"/>
+      <origin xyz="-0.1181 0.01791 -0.09983" rpy="0 0 ${-0.5 * pi}"/>
       <axis xyz="0 0 1"/>
     </joint>
@@ -91,5 +99,5 @@
       <parent link="base_link"/>
       <child link="rotor_arm${child2}"/>
-      <origin xyz="-0.36955 -0.0021 0.045" rpy="0 0 ${pi}"/>
+      <origin xyz="-0.36865 0.0021 0.045" rpy="0 0 ${pi}"/>
       <axis xyz="0 0 1"/>
     </joint>
@@ -206,5 +214,5 @@
       <parent link="rotor_parent${self}"/>
       <child link="thrust${self}"/>
-      <origin rpy="0 0 0" xyz="0 0 0"/>
+      <origin rpy="0 0 0" xyz="0 0 -0.02"/>
       <axis xyz="0 0 ${rotor_direction}"/>
     </joint>
@@ -215,5 +223,5 @@
       <!-- <child link="thrust${self + 2}"/> -->
       <!-- modify this position -->
-      <!-- <origin rpy="0 0 0" xyz="0 0 -0.05"/> -->
+      <!-- <origin rpy="0 0 0" xyz="0 0 -0.02"/> -->
       <!-- <axis xyz="0 0 ${rotor_direction}"/> -->
     <!-- </joint> -->

Commit message: [flamingo][attitude] Enanle reverse rotor thrust for submerge operation

File: robots/flamingo/urdf/flamingo.urdf.xacro (robot description, xacro)
@@ -214,5 +214,5 @@
       <parent link="rotor_parent${self}"/>
       <child link="thrust${self}"/>
-      <origin rpy="0 0 0" xyz="0 0 -0.02"/>
+      <origin rpy="${pi} 0 0" xyz="0 0 -0.02"/>
       <axis xyz="0 0 ${rotor_direction}"/>
     </joint>
