Commit message: Add underwater simulation support for Flamingo robot
- Introduced a new underwater world configuration in
  `aerial_robot_simulation/gazebo_model/world/underwater.world`
  to simulate underwater dynamics with appropriate physics settings.

- Created documentation for underwater simulation in
  `robots/flamingo/doc/underwater_simulation.md`, detailing
  implementation, usage, and parameter tuning.

- Updated `bringup.launch` to support underwater mode, allowing
  seamless switching between aerial and underwater simulations.

- Added `flamingo.gazebo.underwater.xacro` to define the
  Flamingo robot model with underwater hydrodynamics plugin,
  incorporating buoyancy and Fossen model dynamics.

- Modified `flamingo.urdf.xacro` to remove unnecessary inertial
  properties from the root link, simplifying the model for
  underwater simulation.

File: robots/flamingo/urdf/flamingo.urdf.xacro (robot description, xacro)
@@ -4,14 +4,6 @@
   <xacro:macro name="flamingo_center_link" params="child1 child2">
     ## link
-    #### root link (vitrual) ####
-    <link name="root">
-      <inertial>
-        <origin xyz="0 0 0" rpy="0 0 0"/>
-        <mass value="0.00001"/>
-        <inertia
-            ixx="0.000001" iyy="0.000001" izz="0.000001"
-            ixy="0.000000" ixz="0.000000" iyz="0.000000"/>
-      </inertial>
-    </link>
+    #### root link (virtual dummy frame for KDL) ####
+    <link name="root"/>
     #### base link ####
     <link name="base_link">
