Commit message: Revert "Merge upstream "Master" branch into current aerial controller development branch"

File: robots/mini_quadrotor/urdf/robot.urdf.xacro (robot description, xacro)
@@ -96,5 +96,5 @@
   <link name="main_body">
     <inertial>
-      <mass value = "0.860" />
+      <mass value = "0.832" />
       <origin xyz="0.002 0 ${0.028 - 0.002}" rpy="0 0 0"/> <!-- TODO: true cog pos -->
       <inertia
