Commit message: [Nami][urdf] add basci skeleton for nami robot (todo) Modify the pos of each link and use the weight and inertial equal to real machine

File: robots/nami/robots/quad/nami.urdf.xacro (robot description, xacro)
@@ -5,7 +5,7 @@
   <xacro:include filename="$(find nami)/urdf/quad/common.xacro" />
   <xacro:nami_center_link child1="1" child2="2" child3="3" child4="4"/>
-  <xacro:nami_thrust_link self="1" rotor_direction="1"/>
-  <xacro:nami_thrust_link self="2" rotor_direction="-1"/>
-  <xacro:nami_thrust_link self="3" rotor_direction="1"/>
-  <xacro:nami_thrust_link self="4" rotor_direction="-1"/>
+  <xacro:nami_thrust_link_forward self="1" rotor_direction="1"/>
+  <xacro:nami_thrust_link_backward self="2" rotor_direction="-1"/>
+  <xacro:nami_thrust_link_forward self="3" rotor_direction="1"/>
+  <xacro:nami_thrust_link_backward self="4" rotor_direction="-1"/>
 </robot>

File: robots/nami/urdf/quad/nami.urdf.xacro (robot description, xacro)
@@ -1,7 +1,8 @@
 <?xml version="1.0"?>
 <robot
-    xmlns:xacro="http://www.ros.org/wiki/xacro" name="nami_link" >
+    xmlns:xacro="http://www.ros.org/wiki/xacro" name="nami" >
   <xacro:macro name="nami_center_link" params="child1 child2 child3 child4">
-    ## dummy
+    <!-- link -->
+    <!-- root link (virtual) -->
     <link name="root">
       <inertial>
@@ -9,195 +10,369 @@
         <mass value="0.00001"/>
         <inertia
-            ixx="0.000001" ixy="0.0" ixz="0.0"
-            iyy="0.000001" iyz="0.0"
-            izz="0.000001"/>
-      </inertial>
-    </link>
+            ixx="0.000001" iyy="0.000001" izz="0.000001"
+            ixy="0.000000" ixz="0.000000" iyz="0.000000"/>
+      </inertial>
+    </link>
+    <!-- base link head (without spinal on) -->
+    <link name="base_link_head">
+      <inertial>
+      <!-- the relative pos of cog compared to the origin of this link  -->
+      <!-- because right now the origin of base_link has been configured to  the base_link of solidworks-->
+        <origin xyz="0.18668 -0.00002 -0.0409" rpy="0 0 0"/>
+        <mass value="0.89542"/>
+        <inertia
+            ixx="0.0132295" iyy="0.0505483" izz="0.042343"
+            ixy="-0.0000062" ixz="0.0001472" iyz="0.0000005"/>
+      </inertial>
+      <visual>
+        <geometry>
+          <mesh filename="package://nami/urdf/quad/mesh/base_link_head.dae" scale="1 1 1"/>
+          <origin xyz="0.032 -0.01550 0.01850" rpy="0 0 0"/>
+        </geometry>
+      </visual>
+      <collision>
+        <origin xyz="0.18668 -0.00002 -0.0409" rpy="0 0 0"/>
+        <geometry>
+          <box size="0.4045 0.1325 0.2"/>
+        </geometry>
+      </collision>
+    </link>
+    <xacro:damping_factor link="base_link_head"/>
+    <link name="virtual_base_link_tail">
+      <inertial>
+        <origin xyz="0 0 0" rpy="0 0 0"/>
+        <mass value="0.00001"/>
+        <inertia
+            ixx="0.000001" iyy="0.000001" izz="0.000001"
+            ixy="0.000000" ixz="0.000000" iyz="0.000000"/>
+      </inertial>
+    </link>
+    <!-- base link tail (with spinal on top of it) -->
+    <link name="base_link_tail">
+      <inertial>
+        <origin xyz="-0.0782550708 -0.0206739351 0.0236593713" rpy="0 0 0"/>
+        <mass value="2.76613"/>
+        <inertia
+            ixx="0.0132295" iyy="0.0505483" izz="0.042343"
+            ixy="-0.0000062" ixz="0.0001472" iyz="0.0000005"/>
+      </inertial>
+      <visual>
+        <geometry>
+          <mesh filename="package://nami/urdf/quad/mesh/base_link_tail.dae" scale="1 1 1"/>
+          <origin xyz="0.07523 0.02053 0.04926" rpy="0 0 0"/>
+        </geometry>
+      </visual>
+      <collision>
+        <origin xyz="0.0782550708 0.0206739351 0.0236593713"  rpy="0 0 0"/>
+        <geometry>
+          <box size="0.3935 0.1985 0.2"/>
+        </geometry>
+      </collision>
+    </link>
+    <xacro:damping_factor link="base_link_tail"/>
+    <!-- rotor coord link (virtual) -->
+    <link name="rotor_arm${child1}">
+      <inertial>
+        <origin xyz="0 0 0" rpy="0 0 0"/>
+        <mass value="0.00001"/>
+        <inertia
+            ixx="0.000001" iyy="0.000001" izz="0.000001"
+            ixy="0.000000" ixz="0.000000" iyz="0.000000"/>
+      </inertial>
+    </link>
+    <link name="rotor_arm${child2}">
+      <inertial>
+        <origin xyz="0 0 0" rpy="0 0 0"/>
+        <mass value="0.00001"/>
+        <inertia
+            ixx="0.000001" iyy="0.000001" izz="0.000001"
+            ixy="0.000000" ixz="0.000000" iyz="0.000000"/>
+      </inertial>
+    </link>
+    <link name="rotor_arm${child3}">
+      <inertial>
+        <origin xyz="0 0 0" rpy="0 0 0"/>
+        <mass value="0.00001"/>
+        <inertia
+            ixx="0.000001" iyy="0.000001" izz="0.000001"
+            ixy="0.000000" ixz="0.000000" iyz="0.000000"/>
+      </inertial>
+    </link>
+    <link name="rotor_arm${child4}">
+      <inertial>
+        <origin xyz="0 0 0" rpy="0 0 0"/>
+        <mass value="0.00001"/>
+        <inertia
+            ixx="0.000001" iyy="0.000001" izz="0.000001"
+            ixy="0.000000" ixz="0.000000" iyz="0.000000"/>
+      </inertial>
+    </link>
+    <!-- fcu frame -->
+    <link name="fc">
+      <inertial>
+        <origin xyz="0 0 0" rpy="0 0 0"/>
+        <mass value="0.00001"/>
+        <inertia
+            ixx="0.000001" iyy="0.000001" izz="0.000001"
+            ixy="0.000000" ixz="0.000000" iyz="0.000000"/>
+      </inertial>
+    </link>
+    <!-- joints -->
+    <!-- fixed frames (virtual) -->
     <joint name="root_joint" type="fixed">
       <parent link="root"/>
-      <child link="base_link"/>
-      <origin rpy="0 0 0" xyz="0 0 0"/>
-      <axis xyz="0 0 1"/>
-    </joint>
-    ## link
-    <link name="base_link">
-      <inertial>
-        <origin xyz="0.0 0.0 0.0165" rpy="0 0 0"/>
-        <mass value="0.1753"/>
-        <inertia
-            ixx="0.0004" iyy="0.0004" izz="0.0008"
-            ixy="0.00000" ixz="0.0000" iyz="0.00000"/>
-      </inertial>
-      <visual>
-        <origin xyz="0 0 -0.0165" rpy="0 0 0"/>
-        <geometry>
-          <mesh filename="package://nami/urdf/quad/mesh/base_link.STL"/>
-        </geometry>
-      </visual>
-      <collision>
-        <origin xyz="0 0 0" rpy="0 0 0"/>
-        <geometry>
-          <box size="0.25 0.25 0.035"/>
-        </geometry>
-      </collision>
-    </link>
-    <xacro:damping_factor link="base_link"/>
-    <link name="fc">
-      <inertial>
-        <origin xyz="0 0 0" rpy="0 0 0"/>
-        <mass value="0.00001"/>
-        <inertia
-            ixx="0.000001" ixy="0.0" ixz="0.0"
-            iyy="0.000001" iyz="0.0"
-            izz="0.000001"/>
-      </inertial>
-    </link>
+      <child link="base_link_tail"/>
+      <origin xyz="0 0 0" rpy="0 0 0"/>
+    </joint>
     <joint name="fc_joint" type="fixed">
+      <parent link="base_link_tail"/>
       <child link="fc"/>
-      <parent link="base_link"/>
-      <origin rpy="0 0 0" xyz="0 0 0"/>
-      <axis xyz="0 0 1"/>
-    </joint>
-    ## rotor arms
-    <link name="rotor_arm${child1}">
-      <inertial>
-        <origin xyz="0.0486 0 0.0161" rpy="0 0 0"/>
-        <mass value="0.088"/>
-        <inertia
-            ixx="0.000001" ixy="0.0" ixz="0.0"
-            iyy="0.0001" iyz="0.0"
-            izz="0.0001"/>
-      </inertial>
-      <visual>
-        <origin xyz="0 0 0" rpy="0 0 0"/>
-        <geometry>
-          <mesh filename="package://nami/urdf/quad/mesh/rotor_arm.STL"/>
-        </geometry>
-      </visual>
-      <collision>
-        <origin xyz="0 0 0" rpy="0 0 0"/>
-        <geometry>
-          <box size="0.131 0.0325 0.065"/>
-        </geometry>
-      </collision>
-    </link>
-    <joint name="base_arm_joint${child1}" type="fixed">
-      <parent link="base_link"/>
+      <origin xyz="-0.01168 0.02586 0.12094" rpy="0 0 0"/>
+      <axis xyz="0 0 1"/>
+    </joint>
+        <!-- virtual yaw joint of baselink -->
+    <joint name="virtual_yaw_joint" type="fixed">
+      <parent link="base_link_tail"/>
+      <child link="virtual_base_link_tail"/>
+      <origin xyz="0.07523 0.02054 0.02027" rpy="0 0 0"/>
+      <axis xyz="0 0 1"/>
+    </joint>
+    <!-- yaw joint of baselink -->
+    <joint name="yaw_joint" type="revolute">
+      <limit effort="6.6" lower="-1.57" upper="1.57" velocity="3.0"/>
+      <parent link="virtual_base_link_tail"/>
+      <child link="base_link_head"/>
+      <origin xyz="0 0 0" rpy="0 0 0"/>
+      <axis xyz="0 0 1"/>
+      <dynamics damping="0.8" friction="0.0"/>
+    </joint>
+    <!-- rotor coord link joint (virtual) -->
+    <!-- the forward link -->
+    <joint name="rotor_coord_joint${child1}" type="fixed">
+      <parent link="base_link_head" />
       <child link="rotor_arm${child1}"/>
-      <origin rpy="0 0 ${pi/4}" xyz="0.051 0.051 0.0"/>
-      <axis xyz="0 0 1"/>
-    </joint>
-    <link name="rotor_arm${child2}">
-      <inertial>
-        <origin xyz="0.0486 0 0.0161" rpy="0 0 0"/>
-        <mass value="0.088"/>
-        <inertia
-            ixx="0.000001" ixy="0.0" ixz="0.0"
-            iyy="0.0001" iyz="0.0"
-            izz="0.0001"/>
-      </inertial>
-      <visual>
-        <origin xyz="0 0 0" rpy="0 0 0"/>
-        <geometry>
-          <mesh filename="package://nami/urdf/quad/mesh/rotor_arm.STL"/>
-        </geometry>
-      </visual>
-      <collision>
-        <origin xyz="0 0 0" rpy="0 0 0"/>
-        <geometry>
-          <box size="0.131 0.0325 0.065"/>
-        </geometry>p
-      </collision>
-    </link>
-    <joint name="base_arm_joint${child2}" type="fixed">
-      <parent link="base_link"/>
+      <origin xyz="0.2035 0.1825 0.0075" rpy="0 0 0"/>
+      <axis xyz="0 0 1"/>
+    </joint>
+    <joint name="rotor_coord_joint${child2}" type="fixed">
+      <parent link="base_link_head"/>
       <child link="rotor_arm${child2}"/>
-      <origin rpy="0 0 ${pi*3.0/4.0}" xyz="-0.051 0.051 0.0"/>
-      <axis xyz="0 0 1"/>
-    </joint>
-    <link name="rotor_arm${child3}">
-      <inertial>
-        <origin xyz="0.0486 0 0.0161" rpy="0 0 0"/>
-        <mass value="0.088"/>
-        <inertia
-            ixx="0.000001" ixy="0.0" ixz="0.0"
-            iyy="0.0001" iyz="0.0"
-            izz="0.0001"/>
-      </inertial>
-      <visual>
-        <origin xyz="0 0 0" rpy="0 0 0"/>
-        <geometry>
-          <mesh filename="package://nami/urdf/quad/mesh/rotor_arm.STL"/>
-        </geometry>
-      </visual>
-      <collision>
-        <origin xyz="0 0 0" rpy="0 0 0"/>
-        <geometry>
-          <box size="0.131 0.0325 0.065"/>
-        </geometry>
-      </collision>
-    </link>
-    <joint name="base_arm_joint${child3}" type="fixed">
-      <parent link="base_link"/>
+      <origin xyz="0.2035 -0.18327 0.0075" rpy="0 0 ${pi}"/>
+      <axis xyz="0 0 1"/>
+    </joint>
+    <joint name="rotor_coord_joint${child3}" type="fixed">
+      <parent link="base_link_tail"/>
       <child link="rotor_arm${child3}"/>
-      <origin rpy="0 0 ${pi*5.0/4.0}" xyz="-0.051 -0.051 0.0"/>
-      <axis xyz="0 0 1"/>
-    </joint>
-    <link name="rotor_arm${child4}">
-      <inertial>
-        <origin xyz="0.0486 0 0.0161" rpy="0 0 0"/>
-        <mass value="0.088"/>
-        <inertia
-            ixx="0.000001" ixy="0.0" ixz="0.0"
-            iyy="0.0001" iyz="0.0"
-            izz="0.0001"/>
-      </inertial>
-      <visual>
-        <origin xyz="0 0 0" rpy="0 0 0"/>
-        <geometry>
-          <mesh filename="package://nami/urdf/quad/mesh/rotor_arm.STL"/>
-        </geometry>
-      </visual>
-      <collision>
-        <origin xyz="0 0 0" rpy="0 0 0"/>
-        <geometry>
-          <box size="0.131 0.0325 0.065"/>
-        </geometry>
-      </collision>
-    </link>
-    <joint name="base_arm_joint${child4}" type="fixed">
-      <parent link="base_link"/>
+      <origin xyz="-0.14977 -0.16196 0.0277" rpy="0 0 0"/>
+      <axis xyz="0 0 1"/>
+    </joint>
+    <joint name="rotor_coord_joint${child4}" type="fixed">
+      <parent link="base_link_tail"/>
       <child link="rotor_arm${child4}"/>
-      <origin rpy="0 0 ${-pi/4.0}" xyz="0.051 -0.051 0.0"/>
-      <axis xyz="0 0 1"/>
-    </joint>
+      <origin xyz="-0.14977 0.19504 0.0277" rpy="0 0 ${pi}"/>
+      <axis xyz="0 0 1"/>
+    </joint>
+    <!-- gimbal link joint -->
+    <joint name="gimbal${child1}" type="fixed">
+      <limit effort="6.6" lower="-1.57" upper="1.57" velocity="3.0"/>
+      <parent link="rotor_arm${child1}"/>
+      <child link="gimbal_link_forward${child1}"/>
+      <origin xyz="0 0 0" rpy="0 0 ${pi/2}"/>
+      <axis xyz="1 0 0"/>
+      <dynamics damping="0.8" friction="0.0"/>
+    </joint>
+    <joint name="gimbal${child2}" type="fixed">
+      <limit effort="6.6" lower="-1.57" upper="1.57" velocity="3.0"/>
+      <parent link="rotor_arm${child2}"/>
+      <child link="gimbal_link_backward${child2}"/>
+      <origin xyz="0 0 0" rpy="0 0 ${-pi/2}"/>
+      <axis xyz="1 0 0"/>
+      <dynamics damping="0.8" friction="0.0"/>
+    </joint>
+  <joint name="gimbal${child3}" type="fixed">
+      <limit effort="6.6" lower="-1.57" upper="1.57" velocity="3.0"/>
+      <parent link="rotor_arm${child3}"/>
+      <child link="gimbal_link_forward${child3}"/>
+      <origin xyz="0 0 0" rpy="0 0 ${pi/2}"/>
+      <axis xyz="1 0 0"/>
+      <dynamics damping="0.8" friction="0.0"/>
+    </joint>
+    <joint name="gimbal${child4}" type="fixed">
+      <limit effort="6.6" lower="-1.57" upper="1.57" velocity="3.0"/>
+      <parent link="rotor_arm${child4}"/>
+      <child link="gimbal_link_backward${child4}"/>
+      <origin xyz="0 0 0" rpy="0 0 ${-pi/2}"/>
+      <axis xyz="1 0 0"/>
+      <dynamics damping="0.8" friction="0.0"/>
+    </joint>
+    <!-- yaw joint between two body links-->
+    <transmission name="yaw_tran">
+      <type>transmission_interface/SimpleTransmission</type>
+      <joint name="yaw_joint">
+        <hardwareInterface>hardware_interface/EffortJointInterface</hardwareInterface>
+      </joint>
+      <actuator name="servo">
+        <hardwareInterface>hardware_interface/EffortJointInterface</hardwareInterface>
+        <mechanicalReduction>2</mechanicalReduction>
+      </actuator>
+    </transmission>
     <xacro:friction self="base_link"/>
   </xacro:macro>
-  <xacro:macro name="nami_thrust_link" params="self rotor_direction">
-    ## link
-    #### rotor parent link (virtual) ####
-    <link name="gimbal_link${self}">
-      <inertial>
-        <origin xyz="0.018 0.00 0.00438" rpy="0 0 0"/>
-        <mass value="0.1095"/>
-        <inertia
-            ixx="0.00002989" iyy="0.00002848" izz="0.0002698"
-            ixy="0.0000" ixz="-0.0000" iyz="0.00000"/>
-      </inertial>
-      <collision>
-        <origin xyz="0.0 0 0" rpy="0 0 0"/>
-        <geometry>
-          <cylinder radius="0.018" length="0.033"/>
-        </geometry>
-      </collision>
-      <visual>
-        <origin xyz="0 0 0" rpy="0 0 0"/>
-        <geometry>
-          <mesh filename="package://nami/urdf/quad/mesh/rotor_module.STL"/>
-        </geometry>
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