Commit message: [Nami][underwater] surge allocation mode, demo pipeline, and real-machine bringup prep
- NamiController: switchable surge allocation (underwater/surge_allocation):
  rows (Fx, Fz, roll, yaw) instead of legacy (Fz, roll, pitch, yaw); cancels
  the 2.6 N body-x force leak (0.15 -> 0.01 m/s drift in sim A/B), direct
  symmetric surge thrust; pitch passive on the buoyancy righting moment
  (spinal pitch gains zeroed). Legacy allocation kept as default.
- NamiNavigator: underwater/target_depth debug topic for depth plots.
- spinal: port bi-directional PWM support from dev/bi_directional_pwm
  (X3 thrust table, 1.5 ms neutral, 200 Hz, force-landing decay to zero,
  pwm test reverse-range guards) on top of the SIMULATION runtime guards.
- launch: underwater real machine starts ms5837 depth node and disables
  mocap (a started-then-dropped mocap stream trips unhealth level 3
  -> automatic force landing).
- scripts: underwater_demo.py (labeled command sequence + rosbag + chase-cam
  videos), plot_underwater_demo.py, demo_cam/demo_grid models,
  underwater_teleop.py, underwater_flight_test.py.
- docs: allocation DoF analysis, real-machine test checklist, doc updates
  (rotor tilt axis erratum: +-45 deg about body y, not x).

Co-Authored-By: Claude Fable 5 <noreply@anthropic.com>

File: robots/nami/robots/quad/nami.gazebo.underwater.xacro (robot description, xacro)
@@ -4,7 +4,72 @@
   <!-- Standard URDF kinematics -->
   <xacro:include filename="$(find nami)/robots/quad/nami.urdf.xacro" />
+  <!-- ============== Added mass, baked as real inertia (underwater only) ==============
+       The uuv plugin's own <added_mass> computes the force from a numerically
+       differentiated acceleration of the previous step (explicit feedback, EMA
+       alpha=0.3 hard-coded, documented as oscillatory in HydrodynamicModel.cc).
+       Combined with nami's 1e-5 kg virtual thrust links and the yaw_joint two-body
+       coupling it intermittently blows up ODE ("Linear or angular accelerations
+       are invalid" assert), even at scaling 0.1.
+       Instead we bake the added mass into ballast links that gazebo's fixed-joint
+       lumping merges into the two physics bodies: real inertia is handled
+       implicitly by the LCP solver = unconditionally stable. Translational added
+       mass becomes isotropic (mean of the diagonal estimate); rotational added
+       mass is represented exactly by the inertia tensor. The buoyancy volumes in
+       the uuv plugin below are enlarged by dm/rho so the static trim is unchanged
+       (physical added mass carries no weight; here the extra weight and extra
+       buoyancy cancel). Bonus: robot_description mass now includes the added mass,
+       so the controller's force allocation compensates it automatically. -->
+  <!-- tail body: trans diag(0.7 0.9 1.5) -> mean ~1.0 kg; rot diag(0.01 0.02 0.02) -->
+  <link name="added_mass_ballast_tail">
+    <inertial>
+      <origin xyz="0 0 0" rpy="0 0 0"/>
+      <mass value="1.0"/>
+      <inertia ixx="0.01" ixy="0" ixz="0" iyy="0.02" iyz="0" izz="0.02"/>
+    </inertial>
+  </link>
+  <joint name="added_mass_ballast_tail_joint" type="fixed">
+    <parent link="root"/>
+    <child link="added_mass_ballast_tail"/>
+    <!-- at the tail body CoG so the lumped CoG does not move -->
+    <origin xyz="-0.105 0.020 0.023" rpy="0 0 0"/>
+  </joint>
+  <!-- head body: trans diag(0.5 0.6 1.0) -> mean ~0.7 kg; rot diag(0.005 0.015 0.015) -->
+  <link name="added_mass_ballast_head">
+    <inertial>
+      <origin xyz="0 0 0" rpy="0 0 0"/>
+      <mass value="0.7"/>
+      <inertia ixx="0.005" ixy="0" ixz="0" iyy="0.015" iyz="0" izz="0.015"/>
+    </inertial>
+  </link>
+  <joint name="added_mass_ballast_head_joint" type="fixed">
+    <parent link="base_link_head"/>
+    <child link="added_mass_ballast_head"/>
+    <origin xyz="0.194 0.000 -0.022" rpy="0 0 0"/>
+  </joint>
   <!-- Aerial simulation plugin: spinal HW interface, IMU, magnetometer, GPS -->
   <xacro:include filename="$(find aerial_robot_simulation)/xacro/spinal.gazebo.xacro" />
   <xacro:gazebo_spinal robot_name="$(arg robot_name)" mag_frame="fc" />
+  <!-- Depth sensor (uuv_simulator SubseaPressure, model plugin).
+       Publishes sensor_msgs/FluidPressure [kPa] on <robot_namespace>/pressure.
+       Depth is recovered as z = -(P - standard_pressure) / kPa_per_meter (signed, z<0 underwater).
+       link_name must be a physics body that survives fixed-joint reduction, so we use
+       "root" (the tail body containing fc; constant ~0.12 m offset to fc is absorbed
+       because the target depth is initialized from the current reading).
+       noise_sigma/amplitude start at 0 for clean bring-up - add noise when tuning. -->
+  <gazebo>
+    <plugin name="subsea_pressure_plugin" filename="libuuv_gazebo_ros_subsea_pressure_plugin.so">
+      <robot_namespace>$(arg robot_name)</robot_namespace>
+      <link_name>root</link_name>
+      <sensor_topic>pressure</sensor_topic>
+      <update_rate>50</update_rate>
+      <saturation>3000</saturation>
+      <noise_sigma>0.0</noise_sigma>
+      <noise_amplitude>0.0</noise_amplitude>
+      <estimate_depth_on>false</estimate_depth_on>
+      <standard_pressure>101.325</standard_pressure>
+      <kPa_per_meter>9.80638</kPa_per_meter>
+      <enable_gazebo_messages>false</enable_gazebo_messages>
+    </plugin>
+  </gazebo>
   <!-- Underwater hydrodynamics plugin (uuv_simulator).
        Applies buoyancy + Fossen-model hydrodynamic forces to the listed links each
@@ -37,11 +102,12 @@
       <debug>0</debug>
       <!-- ================= tail-side body (physics body "root") =================
-           mass 2.355 kg -> neutral volume 0.002355 m^3 in freshwater.
-           volume set ~1% above neutral for slight positive buoyancy (~0.25 N up).
+           mass 2.355 kg + 1.0 kg baked added-mass ballast = 3.355 kg
+           -> neutral volume 0.003355 m^3 in freshwater; set ~1% above neutral
+           for slight positive buoyancy (~0.35 N up).
            WARNING: buoyancy applies only while the link is below z=0, and the
            robot is ejected to the surface if volume is set far above neutral. -->
       <link name="root">
         <neutrally_buoyant>0</neutrally_buoyant>
-        <volume>0.00238</volume>
+        <volume>0.00349</volume>
         <!-- Bounding box used only for debug visualisation; no effect on forces -->
         <box>
@@ -57,20 +123,22 @@
         <hydrodynamic_model>
           <type>fossen</type>
-          <!-- Added mass [kg, kg*m^2] - 6x6 row-major, diagonal approximation.
-               Translational ~30% of displaced mass (heave larger: flat body +
-               two rotor discs). Rotational terms kept small. Refine by system
-               identification. -->
+          <!-- Added mass: kept ZERO here. The plugin computes it from a numerically
+               differentiated acceleration (explicit feedback) which intermittently
+               NaN-crashed ODE even at scaling 0.1. The physical added mass
+               (trans diag(0.7 0.9 1.5), rot diag(0.01 0.02 0.02)) is baked into the
+               added_mass_ballast_tail link instead - see the note at the top. -->
           <added_mass>
-             0.7  0    0    0    0    0
-             0    0.9  0    0    0    0
-             0    0    1.5  0    0    0
-             0    0    0    0.01 0    0
-             0    0    0    0    0.02 0
-             0    0    0    0    0    0.02
+             0 0 0 0 0 0
+             0 0 0 0 0 0
+             0 0 0 0 0 0
+             0 0 0 0 0 0
+             0 0 0 0 0 0
+             0 0 0 0 0 0
           </added_mass>
           <!-- Linear damping [N*s/m, N*m*s/rad] - diagonal 6-vector.
-               Stokes-drag scale; mainly suppresses slow drift. -->
+               Raised from the pure Stokes estimate to damp the added-mass
+               feedback oscillation (see note above). -->
           <linear_damping>
-            -5 -5 -10 -0.5 -0.5 -0.5
+            -8 -8 -15 -0.8 -0.8 -0.8
           </linear_damping>
           <!-- Quadratic damping [N*s^2/m^2, N*m*s^2/rad^2] - diagonal 6-vector.
@@ -85,8 +153,9 @@
       </link>
       <!-- ================= head-side body ("base_link_head") =================
-           mass 1.600 kg -> neutral volume 0.001600 m^3; set ~1% above. -->
+           mass 1.600 kg + 0.7 kg baked added-mass ballast = 2.300 kg
+           -> neutral volume 0.002300 m^3; set ~1% above. -->
       <link name="base_link_head">
         <neutrally_buoyant>0</neutrally_buoyant>
-        <volume>0.00162</volume>
+        <volume>0.002329</volume>
         <box>
           <width>0.133</width>
@@ -99,11 +168,14 @@
         <hydrodynamic_model>
           <type>fossen</type>
+          <!-- kept ZERO: the physical added mass (trans diag(0.5 0.6 1.0),
+               rot diag(0.005 0.015 0.015)) is baked into added_mass_ballast_head
+               as real inertia - see the note at the top. -->
           <added_mass>
-             0.5  0    0    0    0    0
-             0    0.6  0    0    0    0
-             0    0    1.0  0    0    0
-             0    0    0    0.005 0    0
-             0    0    0    0    0.015 0
-             0    0    0    0    0    0.015
+             0 0 0 0 0 0
+             0 0 0 0 0 0
+             0 0 0 0 0 0
+             0 0 0 0 0 0
+             0 0 0 0 0 0
+             0 0 0 0 0 0
           </added_mass>
           <linear_damping>

File: robots/nami/robots/quad/nami.urdf.xacro (robot description, xacro)
@@ -9,3 +9,8 @@
   <xacro:nami_thrust_link_forward self="3" rotor_direction="1"/>
   <xacro:nami_thrust_link_backward self="4" rotor_direction="-1"/>
+  <!-- aquatic actuators: logical motor 4~7 (thrust5..8), used only in underwater mode -->
+  <xacro:nami_aquatic_actuator self="1" motor_id="5" rotor_direction="1"/>
+  <xacro:nami_aquatic_actuator self="2" motor_id="6" rotor_direction="-1"/>
+  <xacro:nami_aquatic_actuator self="3" motor_id="7" rotor_direction="1"/>
+  <xacro:nami_aquatic_actuator self="4" motor_id="8" rotor_direction="-1"/>
 </robot>

File: robots/nami/urdf/quad/common.xacro (robot description, xacro)
@@ -8,4 +8,8 @@
   <xacro:property name="max_force" value="18.2494" /> <!-- [N] -->
   <xacro:property name="min_force" value="1.0" /> <!-- [N] -->
+  <!-- aquatic rotor (ApiSqueen X3, 24V): asymmetric bi-directional thrust range,
+       endpoints taken from the convertBiDirectional table in dev/bi_directional_pwm -->
+  <xacro:property name="aquatic_max_forward_force" value="25.48" /> <!-- [N] -->
+  <xacro:property name="aquatic_max_reverse_force" value="14.7" /> <!-- [N] -->
   <!-- friction -->
   <xacro:macro name="friction" params="self">

File: robots/nami/urdf/quad/nami.urdf.xacro (robot description, xacro)
@@ -281,11 +281,15 @@
       </inertial>
     </link>
-    <!-- thrust link (virtual) -->
+    <!-- thrust link (virtual).
+         0.01 kg instead of the usual 1e-5: even force-free, a 1e-5 kg body on a
+         continuous joint sits in the same ODE constraint island as the ~3 kg hydro
+         bodies underwater and the extreme mass ratio intermittently NaNs the LCP
+         solve (see the aquatic thrust link note). -->
     <link name="thrust${self}">
       <inertial>
         <origin xyz="0 0 0" rpy="0 0 0"/>
-        <mass value="0.00001"/>
-        <inertia
-            ixx="0.000001" iyy="0.000001" izz="0.000001"
+        <mass value="0.01"/>
+        <inertia
+            ixx="0.00001" iyy="0.00001" izz="0.00001"
             ixy="0.000000" ixz="0.000000" iyz="0.000000"/>
       </inertial>
@@ -381,11 +385,15 @@
       </inertial>
     </link>
-    <!-- thrust link (virtual) -->
+    <!-- thrust link (virtual).
+         0.01 kg instead of the usual 1e-5: even force-free, a 1e-5 kg body on a
+         continuous joint sits in the same ODE constraint island as the ~3 kg hydro
+         bodies underwater and the extreme mass ratio intermittently NaNs the LCP
+         solve (see the aquatic thrust link note). -->
     <link name="thrust${self}">
       <inertial>
         <origin xyz="0 0 0" rpy="0 0 0"/>
-        <mass value="0.00001"/>
-        <inertia
-            ixx="0.000001" iyy="0.000001" izz="0.000001"
+        <mass value="0.01"/>
+        <inertia
+            ixx="0.00001" iyy="0.00001" izz="0.00001"
             ixy="0.000000" ixz="0.000000" iyz="0.000000"/>
       </inertial>
@@ -432,3 +440,61 @@
     </transmission>
   </xacro:macro>
+  <!-- aquatic rotor actuator (logical motor ${motor_id} = unit ${self} + 4).
+       Thrust acts along the z axis of aquatic_rotor${self} (tilted +-45 deg about x).
+       Bi-directional: joint limit lower is negative so the gazebo rotor saturation
+       (EffortRotorSaturationHandle) admits reverse thrust; on the real machine these
+       map to motor 4~7 on pwm_htim2 (dev/bi_directional_pwm, 1500us neutral). -->
+  <xacro:macro name="nami_aquatic_actuator" params="self motor_id rotor_direction">
+    <!-- rotor parent link (virtual) -->
+    <link name="rotor_parent_aquatic${self}">
+      <inertial>
+        <origin xyz="0 0 0" rpy="0 0 0"/>
+        <mass value="0.00001"/>
+        <inertia
+            ixx="0.000001" iyy="0.000001" izz="0.000001"
+            ixy="0.000000" ixz="0.000000" iyz="0.000000"/>
+      </inertial>
+    </link>
+    <joint name="rotor_parent_aquatic_joint${self}" type="fixed">
+      <parent link="aquatic_rotor${self}"/>
+      <child link="rotor_parent_aquatic${self}"/>
+      <origin xyz="0 0 0" rpy="0 0 0"/>
+    </joint>
+    <!-- thrust link (virtual).
+         NOT the usual 1e-5 kg: these links take the full bi-directional aquatic
+         thrust (up to ~25 N) while the parent bodies carry large hydrodynamic
+         forces underwater. A 1e-5 kg link gives ODE a ~1:3e5 mass ratio in the
+         constraint island, which intermittently fails the LCP solve and NaN-crashes
+         gazebo (uuv plugin acceleration assert). 0.01 kg keeps the physics healthy
+         and only adds 40 g to the model. -->
+    <link name="thrust${motor_id}">
+      <inertial>
+        <origin xyz="0 0 0" rpy="0 0 0"/>
+        <mass value="0.01"/>
+        <inertia
+            ixx="0.00001" iyy="0.00001" izz="0.00001"
+            ixy="0.000000" ixz="0.000000" iyz="0.000000"/>
+      </inertial>
+    </link>
+    <xacro:damping_factor link="thrust${motor_id}"/>
+    <!-- rotor joint (virtual): asymmetric bi-directional force range -->
+    <joint name="rotor${motor_id}" type="continuous">
+      <limit effort="100.0" lower="-${aquatic_max_reverse_force}" upper="${aquatic_max_forward_force}" velocity="0.5"/>
+      <parent link="rotor_parent_aquatic${self}"/>
+      <child link="thrust${motor_id}"/>
+      <origin rpy="0 0 0" xyz="0 0 0"/>
+      <axis xyz="0 0 ${rotor_direction}"/>
+    </joint>
+    <!-- hardware interface -->
+    <transmission name="rotor_tran${motor_id}">
+      <type>transmission_interface/SimpleTransmission</type>
+      <joint name="rotor${motor_id}">
+        <hardwareInterface>RotorInterface</hardwareInterface>
+      </joint>
+      <actuator name="rotor_actuator${motor_id}">
+        <hardwareInterface>RotorInterface</hardwareInterface>
+        <mechanicalReduction>1</mechanicalReduction>
+      </actuator>
+    </transmission>
+  </xacro:macro>
 </robot>
