Commit message: [Nami][urdf] Update Nami URDF parameters: refine mass, inertia, and joint origin values

File: robots/nami/urdf/quad/common.xacro (robot description, xacro)
@@ -5,6 +5,6 @@
   <baselink name="fc" />
   <thrust_link name="thrust" />
-  <m_f_rate value="-0.0172" /> <!-- drug torque rate -->
-  <xacro:property name="max_force" value="18.0" /> <!-- [N] -->
+  <m_f_rate value="-0.0068" /> <!-- drug torque rate -->
+  <xacro:property name="max_force" value="18.2494" /> <!-- [N] -->
   <xacro:property name="min_force" value="1.0" /> <!-- [N] -->
   <!-- friction -->

File: robots/nami/urdf/quad/nami.urdf.xacro (robot description, xacro)
@@ -19,9 +19,9 @@
       <!-- the relative pos of cog compared to the origin of this link  -->
       <!-- because right now the origin of base_link has been configured to  the base_link of solidworks-->
-        <origin xyz="0.18668 -0.00002 -0.0409" rpy="0 0 0"/>
-        <mass value="0.89542"/>
-        <inertia
-            ixx="0.0132295" iyy="0.0505483" izz="0.042343"
-            ixy="-0.0000062" ixz="0.0001472" iyz="0.0000005"/>
+        <origin xyz="0.186933 -0.000016 -0.042086" rpy="0 0 0"/>
+        <mass value="0.940089"/>
+        <inertia
+            ixx="0.001164" iyy="0.006858" izz="0.006443"
+            ixy="-0.000002" ixz="-0.000515" iyz="0.000001"/>
       </inertial>
       <visual>
@@ -31,6 +31,6 @@
         </geometry>
       </visual>
-      <collision>
-        <origin xyz="0.18668 -0.00002 -0.0409" rpy="0 0 0"/>
+      <collision>`
+        <origin xyz="0.186933 -0.000016 -0.042086" rpy="0 0 0"/>
         <geometry>
           <box size="0.4045 0.1325 0.2"/>
@@ -51,9 +51,9 @@
     <link name="base_link_tail">
       <inertial>
-        <origin xyz="-0.0782550708 -0.0206739351 0.0236593713" rpy="0 0 0"/>
-        <mass value="2.76613"/>
-        <inertia
-            ixx="0.0132295" iyy="0.0505483" izz="0.042343"
-            ixy="-0.0000062" ixz="0.0001472" iyz="0.0000005"/>
+        <origin xyz="-0.0811138 0.02019128 0.0206661" rpy="0 0 0"/>
+        <mass value="1.6950211"/>
+        <inertia
+            ixx="0.0080266" iyy="0.0245560" izz="0.0188846"
+            ixy="-0.0000106" ixz="0.0062218" iyz="-0.0000356"/>
       </inertial>
       <visual>
@@ -64,5 +64,5 @@
       </visual>
       <collision>
-        <origin xyz="0.0782550708 0.0206739351 0.0236593713"  rpy="0 0 0"/>
+        <origin xyz="-0.0811138 0.02019128 0.0206661"  rpy="0 0 0"/>
         <geometry>
           <box size="0.3935 0.1985 0.2"/>
@@ -128,5 +128,5 @@
       <parent link="base_link_tail"/>
       <child link="fc"/>
-      <origin xyz="-0.0183192 0.02586 0.12004" rpy="0 0 0"/>
+      <origin xyz="0.0183193 0.0284366 0.1200359" rpy="0 0 0"/>
       <axis xyz="0 0 1"/>
     </joint>
@@ -222,9 +222,9 @@
     <!-- this link's cordinate is the actual gimbal -->
       <inertial>
-        <origin xyz="0.0328427 -0.0000782 -0.0167858" rpy="0 0 0"/>
-        <mass value="0.27076"/>
-        <inertia
-            ixx="0.0007257" iyy="0.0007451" izz="0.0000987"
-            ixy="0.0000007" ixz="-0.0000189" iyz="-0.0000001"/>
+        <origin xyz="-0.011008 0.000169 0.023330" rpy="0 0 0"/>
+        <mass value="0.186457"/>
+        <inertia
+            ixx="0.000201" iyy="0.000347" izz="0.000450"
+            ixy="-0.000002" ixz="0.000004" iyz="0.000000"/>
       </inertial>
       <visual>
@@ -235,5 +235,5 @@
       </visual>
       <collision>
-        <origin xyz="0.036 0 -0.006" rpy="0 0 0"/>
+        <origin xyz="-0.011008 0.000169 0.023330" rpy="0 0 0"/>
         <geometry>
           <cylinder radius="0.12662" length="0.1578"/>
@@ -246,9 +246,9 @@
     <!-- this link's cordinate is the actual gimbal -->
       <inertial>
-        <origin xyz="0.0328427 -0.0000782 -0.0167858" rpy="0 0 0"/>
-        <mass value="0.27076"/>
-        <inertia
-            ixx="0.0007257" iyy="0.0007451" izz="0.0000987"
-            ixy="0.0000007" ixz="-0.0000189" iyz="-0.0000001"/>
+        <origin xyz="0.001352 -0.000410 -0.045541" rpy="0 0 0"/>
+        <mass value="0.14360"/>
+        <inertia
+            ixx="0.000227" iyy="0.000224" izz="0.000037"
+            ixy="0.000000" ixz="-0.000003" iyz="0.000001"/>
       </inertial>
       <visual>
@@ -259,5 +259,5 @@
       </visual>
       <collision>
-        <origin xyz="0.036 0 -0.006" rpy="0 0 0"/>
+        <origin xyz="0.001352 -0.000410 -0.045541" rpy="0 0 0"/>
         <geometry>
           <cylinder radius="0.12662" length="0.1578"/>
@@ -328,9 +328,9 @@
     <!-- this link's cordinate is the actual gimbal -->
       <inertial>
-        <origin xyz="0.0328427 -0.0000782 -0.0167858" rpy="0 0 0"/>
-        <mass value="0.27076"/>
-        <inertia
-            ixx="0.0007257" iyy="0.0007451" izz="0.0000987"
-            ixy="0.0000007" ixz="-0.0000189" iyz="-0.0000001"/>
+        <origin xyz="-0.011008 0.000169 0.023330" rpy="0 0 0"/>
+        <mass value="0.186457"/>
+        <inertia
+            ixx="0.000201" iyy="0.000347" izz="0.000450"
+            ixy="-0.000002" ixz="0.000004" iyz="0.000000"/>
       </inertial>
       <visual>
@@ -341,5 +341,5 @@
       </visual>
       <collision>
-        <origin xyz="0.036 0 -0.006" rpy="0 0 0"/>
+        <origin xyz="-0.011008 0.000169 0.023330" rpy="0 0 0"/>
         <geometry>
           <cylinder radius="0.12662" length="0.1578"/>
@@ -352,9 +352,9 @@
     <!-- this link's cordinate is the actual gimbal -->
       <inertial>
-        <origin xyz="0.0328427 -0.0000782 -0.0167858" rpy="0 0 0"/>
-        <mass value="0.27076"/>
-        <inertia
-            ixx="0.0007257" iyy="0.0007451" izz="0.0000987"
-            ixy="0.0000007" ixz="-0.0000189" iyz="-0.0000001"/>
+        <origin xyz="0.001352 -0.000410 -0.045541" rpy="0 0 0"/>
+        <mass value="0.14360"/>
+        <inertia
+            ixx="0.000227" iyy="0.000224" izz="0.000037"
+            ixy="0.000000" ixz="-0.000003" iyz="0.000001"/>
       </inertial>
       <visual>
@@ -365,5 +365,5 @@
       </visual>
       <collision>
-        <origin xyz="0.036 0 -0.006" rpy="0 0 0"/>
+        <origin xyz="0.001352 -0.000410 -0.045541" rpy="0 0 0"/>
         <geometry>
           <cylinder radius="0.12662" length="0.1578"/>
