Commit message: [Nami][urdf] Refactor Nami URDF Xacro: Update joint origins and inertia parameters for improved accuracy
- Adjusted the origin positions for the `fc_joint` and `virtual_yaw_joint` to enhance alignment.
- Updated inertia parameters for various links to reflect more accurate physical properties.
- Refined the joint configurations for rotor arms to ensure proper attachment and movement.
- Added damping factors for thrust links to improve simulation stability.
- Ensured consistent naming conventions and formatting throughout the file.

File: robots/nami/urdf/quad/nami.urdf.xacro (robot description, xacro)
@@ -26,7 +26,7 @@
       </inertial>
       <visual>
+        <origin xyz="0.032 -0.01550 0.01850" rpy="0 0 0"/>
         <geometry>
           <mesh filename="package://nami/urdf/quad/mesh/base_link_head.dae" scale="1 1 1"/>
-          <origin xyz="0.032 -0.01550 0.01850" rpy="0 0 0"/>
         </geometry>
       </visual>
@@ -58,7 +58,7 @@
       </inertial>
       <visual>
+        <origin xyz="0.07523 0.02053 0.04926" rpy="0 0 0"/>
         <geometry>
           <mesh filename="package://nami/urdf/quad/mesh/base_link_tail.dae" scale="1 1 1"/>
-          <origin xyz="0.07523 0.02053 0.04926" rpy="0 0 0"/>
         </geometry>
       </visual>
@@ -128,5 +128,5 @@
       <parent link="base_link_tail"/>
       <child link="fc"/>
-      <origin xyz="-0.01168 0.02586 0.12094" rpy="0 0 0"/>
+      <origin xyz="-0.0183192 0.02586 0.12004" rpy="0 0 0"/>
       <axis xyz="0 0 1"/>
     </joint>
@@ -136,5 +136,4 @@
       <child link="virtual_base_link_tail"/>
       <origin xyz="0.07523 0.02054 0.02027" rpy="0 0 0"/>
-      <axis xyz="0 0 1"/>
     </joint>
     <!-- yaw joint of baselink -->
@@ -158,5 +157,5 @@
       <parent link="base_link_head"/>
       <child link="rotor_arm${child2}"/>
-      <origin xyz="0.2035 -0.18327 0.0075" rpy="0 0 ${pi}"/>
+      <origin xyz="0.2035 -0.1825 0.0075" rpy="0 0 0"/>
       <axis xyz="0 0 1"/>
     </joint>
@@ -164,5 +163,5 @@
       <parent link="base_link_tail"/>
       <child link="rotor_arm${child3}"/>
-      <origin xyz="-0.14977 -0.16196 0.0277" rpy="0 0 0"/>
+      <origin xyz="-0.16627 -0.16196 0.02777" rpy="0 0 0"/>
       <axis xyz="0 0 1"/>
     </joint>
@@ -170,5 +169,5 @@
       <parent link="base_link_tail"/>
       <child link="rotor_arm${child4}"/>
-      <origin xyz="-0.14977 0.19504 0.0277" rpy="0 0 ${pi}"/>
+      <origin xyz="-0.16627 0.20304 0.02777" rpy="0 0 0"/>
       <axis xyz="0 0 1"/>
     </joint>
@@ -179,6 +178,5 @@
       <child link="gimbal_link_forward${child1}"/>
       <origin xyz="0 0 0" rpy="0 0 ${pi/2}"/>
-      <axis xyz="1 0 0"/>
-      <dynamics damping="0.8" friction="0.0"/>
+      <axis xyz="0 0 1"/>
     </joint>
     <joint name="gimbal${child2}" type="fixed">
@@ -187,6 +185,5 @@
       <child link="gimbal_link_backward${child2}"/>
       <origin xyz="0 0 0" rpy="0 0 ${-pi/2}"/>
-      <axis xyz="1 0 0"/>
-      <dynamics damping="0.8" friction="0.0"/>
+      <axis xyz="0 0 1"/>
     </joint>
   <joint name="gimbal${child3}" type="fixed">
@@ -194,7 +191,6 @@
       <parent link="rotor_arm${child3}"/>
       <child link="gimbal_link_forward${child3}"/>
-      <origin xyz="0 0 0" rpy="0 0 ${pi/2}"/>
-      <axis xyz="1 0 0"/>
-      <dynamics damping="0.8" friction="0.0"/>
+      <origin xyz="0 0 0" rpy="0 0 ${-pi/2}"/>
+      <axis xyz="0 0 1"/>
     </joint>
     <joint name="gimbal${child4}" type="fixed">
@@ -202,7 +198,6 @@
       <parent link="rotor_arm${child4}"/>
       <child link="gimbal_link_backward${child4}"/>
-      <origin xyz="0 0 0" rpy="0 0 ${-pi/2}"/>
-      <axis xyz="1 0 0"/>
-      <dynamics damping="0.8" friction="0.0"/>
+      <origin xyz="0 0 0" rpy="0 0 ${pi/2}"/>
+      <axis xyz="0 0 1"/>
     </joint>
     <!-- yaw joint between two body links-->
@@ -217,5 +212,6 @@
       </actuator>
     </transmission>
-    <xacro:friction self="base_link"/>
+    <xacro:friction self="base_link_head"/>
+    <xacro:friction self="base_link_tai"/>
   </xacro:macro>
   <xacro:macro name="nami_thrust_link_forward" params="self rotor_direction">
@@ -271,5 +267,5 @@
       <parent link="gimbal_link_forward${self}"/>
       <child link="aquatic_rotor${self}"/>
-      <origin xyz="-0.0755 -0.0396 -0.0176" rpy="${3*pi/2} 0 0"/>
+      <origin xyz="-0.0755 -0.0396 -0.0176" rpy="${-pi/4} 0 0"/>
       <axis xyz="1 0 0"/>
     </joint>
@@ -375,5 +371,5 @@
     </link>
     <!-- rotor parent link (virtual) -->
-    <link name="rotor_parent${self}">
+    <link name="rotor_parent_backward${self}">
       <inertial>
         <origin xyz="0 0 0" rpy="0 0 0"/>
@@ -398,5 +394,5 @@
       <parent link="gimbal_link_backward${self}"/>
       <child link="aquatic_rotor${self}"/>
-      <origin xyz="-0.0755 0.0396 -0.0176" rpy="${-3*pi/2} 0 0"/>
+      <origin xyz="-0.0755 0.0396 -0.0176" rpy="${pi/4} 0 0"/>
       <axis xyz="1 0 0"/>
     </joint>
@@ -405,5 +401,5 @@
     <joint name="rotor_parent_link_joint${self}" type="fixed">
       <parent link="gimbal_link_backward${self}"/>
-      <child link="rotor_parent${self}"/>
+      <child link="rotor_parent_backward${self}"/>
       <origin xyz="0 0 0" rpy="0 0 0"/>
       <axis xyz="0 0 1"/>
@@ -417,5 +413,5 @@
     <!-- should change the min and max force in motor_info.yaml file -->
       <limit effort="100.0" lower="${min_force}" upper="${max_force}" velocity="0.5"/>
-      <parent link="rotor_parent${self}"/>
+      <parent link="rotor_parent_backward${self}"/>
       <child link="thrust${self}"/>
       <origin rpy="0 0 0" xyz="0 0 0"/>

Commit message: [Nami][launch] Update robot_id in mocap.launch; [Nami][config] Enable DSHOT in config.h; [Nami][config] Adjust zero_point_offset in Servo.yaml; [Nami][launch] Lock yaw joint servo at zero point in bringup.launch; [Nami][urdf] Modify fc_joint origin in nami.urdf.xacro

File: robots/nami/urdf/quad/nami.urdf.xacro (robot description, xacro)
@@ -128,5 +128,5 @@
       <parent link="base_link_tail"/>
       <child link="fc"/>
-      <origin xyz="0.0183193 0.0284366 0.1200359" rpy="0 0 0"/>
+      <origin xyz="0.0183193 0.0284366 0.1300359" rpy="0 0 0"/>
       <axis xyz="0 0 1"/>
     </joint>

Commit message: [Nami][urdf] Update inertial parameters for base link tail: adjust origin and inertia values for improved accuracy

File: robots/nami/urdf/quad/nami.urdf.xacro (robot description, xacro)
@@ -51,9 +51,9 @@
     <link name="base_link_tail">
       <inertial>
-        <origin xyz="-0.0811138 0.02019128 0.0206661" rpy="0 0 0"/>
+        <origin xyz="-0.0169110 0.0200899 0.0630640" rpy="0 0 0"/>
         <mass value="1.6950211"/>
         <inertia
-            ixx="0.0080266" iyy="0.0245560" izz="0.0188846"
-            ixy="-0.0000106" ixz="0.0062218" iyz="-0.0000356"/>
+            ixx="0.0040010" iyy="0.0098791" izz="0.0076315"
+            ixy="0.0000156" ixz="0.0004014" iyz="-0.0000250"/>
       </inertial>
       <visual>
@@ -64,5 +64,5 @@
       </visual>
       <collision>
-        <origin xyz="-0.0811138 0.02019128 0.0206661"  rpy="0 0 0"/>
+        <origin xyz="-0.0169110 0.0200899 0.0630640"  rpy="0 0 0"/>
         <geometry>
           <box size="0.3935 0.1985 0.2"/>

Commit message: [Update] adjust rotor coordinate joint origins for improved alignment

File: robots/nami/urdf/quad/nami.urdf.xacro (robot description, xacro)
@@ -52,5 +52,5 @@
       <inertial>
         <origin xyz="-0.0169110 0.0200899 0.0630640" rpy="0 0 0"/>
-        <mass value="1.6950211"/>
+        <mass value="1.073"/>
         <inertia
             ixx="0.0040010" iyy="0.0098791" izz="0.0076315"
@@ -152,5 +152,5 @@
       <parent link="base_link_head" />
       <child link="rotor_arm${child1}"/>
-      <origin xyz="0.2035 0.1825 0.0075" rpy="0 0 0"/>
+      <origin xyz="0.2105 0.1945 0.007" rpy="0 0 0"/>
       <axis xyz="0 0 1"/>
     </joint>
@@ -158,5 +158,5 @@
       <parent link="base_link_head"/>
       <child link="rotor_arm${child2}"/>
-      <origin xyz="0.2035 -0.1825 0.0075" rpy="0 0 0"/>
+      <origin xyz="0.2105 -0.2025 0.007" rpy="0 0 0"/>
       <axis xyz="0 0 1"/>
     </joint>
@@ -164,5 +164,5 @@
       <parent link="base_link_tail"/>
       <child link="rotor_arm${child3}"/>
-      <origin xyz="-0.16627 -0.16196 0.02777" rpy="0 0 0"/>
+      <origin xyz="-0.20427 -0.18336 0.02777" rpy="0 0 0"/>
       <axis xyz="0 0 1"/>
     </joint>
@@ -170,5 +170,5 @@
       <parent link="base_link_tail"/>
       <child link="rotor_arm${child4}"/>
-      <origin xyz="-0.16627 0.20304 0.02777" rpy="0 0 0"/>
+      <origin xyz="-0.20427 0.22304 0.02777" rpy="0 0 0"/>
       <axis xyz="0 0 1"/>
     </joint>

Commit message: [Update] adjust PID gains and mass properties for improved underwater control dynamics

File: robots/nami/urdf/quad/nami.urdf.xacro (robot description, xacro)
@@ -20,5 +20,5 @@
       <!-- because right now the origin of base_link has been configured to  the base_link of solidworks-->
         <origin xyz="0.186933 -0.000016 -0.042086" rpy="0 0 0"/>
-        <mass value="0.940089"/>
+        <mass value="0.520089"/>
         <inertia
             ixx="0.001164" iyy="0.006858" izz="0.006443"
@@ -128,5 +128,5 @@
       <parent link="base_link_tail"/>
       <child link="fc"/>
-      <origin xyz="0.0183193 0.0284366 0.1300359" rpy="0 0 0"/>
+      <origin xyz="0.0183193 0.0284366 0.1300359" rpy="0 0 ${pi}"/>
       <axis xyz="0 0 1"/>
     </joint>

Commit message: [Update] update the URDF model parameters for square version of nami

File: robots/nami/urdf/quad/nami.urdf.xacro (robot description, xacro)
@@ -19,9 +19,9 @@
       <!-- the relative pos of cog compared to the origin of this link  -->
       <!-- because right now the origin of base_link has been configured to  the base_link of solidworks-->
-        <origin xyz="0.186933 -0.000016 -0.042086" rpy="0 0 0"/>
-        <mass value="0.520089"/>
-        <inertia
-            ixx="0.001164" iyy="0.006858" izz="0.006443"
-            ixy="-0.000002" ixz="-0.000515" iyz="0.000001"/>
+        <origin xyz="0.221545 -0.000011 -0.042583" rpy="0 0 0"/>
+        <mass value="0.940089"/>
+        <inertia
+            ixx="0.001302" iyy="0.009489" izz="0.00899"
+            ixy="-0.000002" ixz="-0.000632" iyz="0.000001"/>
       </inertial>
       <visual>
@@ -31,6 +31,6 @@
         </geometry>
       </visual>
-      <collision>`
-        <origin xyz="0.186933 -0.000016 -0.042086" rpy="0 0 0"/>
+      <collision>
+        <origin xyz="0.221545 -0.000011 -0.042583" rpy="0 0 0"/>
         <geometry>
           <box size="0.4045 0.1325 0.2"/>
@@ -51,12 +51,12 @@
     <link name="base_link_tail">
       <inertial>
-        <origin xyz="-0.0169110 0.0200899 0.0630640" rpy="0 0 0"/>
+        <origin xyz="-0.0647393 0.0516416 0.0854933" rpy="0 0 0"/>
         <mass value="1.073"/>
         <inertia
-            ixx="0.0040010" iyy="0.0098791" izz="0.0076315"
-            ixy="0.0000156" ixz="0.0004014" iyz="-0.0000250"/>
+            ixx="0.0043312" iyy="0.0132108" izz="0.0110638"
+            ixy="0.0000063" ixz="0.001385" iyz="-0.0000162"/>
       </inertial>
       <visual>
-        <origin xyz="0.07523 0.02053 0.04926" rpy="0 0 0"/>
+        <origin xyz="-0.0647393 0.0516416 0.0854933" rpy="0 0 0"/>
         <geometry>
           <mesh filename="package://nami/urdf/quad/mesh/base_link_tail.dae" scale="1 1 1"/>
@@ -128,5 +128,5 @@
       <parent link="base_link_tail"/>
       <child link="fc"/>
-      <origin xyz="0.0183193 0.0284366 0.1300359" rpy="0 0 ${pi}"/>
+      <origin xyz="0.01895 0.0599 0.13886" rpy="0 0 0"/>
       <axis xyz="0 0 1"/>
     </joint>
@@ -135,5 +135,5 @@
       <parent link="base_link_tail"/>
       <child link="virtual_base_link_tail"/>
-      <origin xyz="0.07523 0.02054 0.02027" rpy="0 0 0"/>
+      <origin xyz="0.03797 0.052 0.02909" rpy="0 0 0"/>
     </joint>
     <!-- yaw joint of baselink -->
@@ -152,5 +152,5 @@
       <parent link="base_link_head" />
       <child link="rotor_arm${child1}"/>
-      <origin xyz="0.2105 0.1945 0.007" rpy="0 0 0"/>
+      <origin xyz="0.2285 0.2025 0.0045" rpy="0 0 0"/>
       <axis xyz="0 0 1"/>
     </joint>
@@ -158,5 +158,5 @@
       <parent link="base_link_head"/>
       <child link="rotor_arm${child2}"/>
-      <origin xyz="0.2105 -0.2025 0.007" rpy="0 0 0"/>
+      <origin xyz="0.2285 -0.2025 0.0045" rpy="0 0 0"/>
       <axis xyz="0 0 1"/>
     </joint>
@@ -164,5 +164,5 @@
       <parent link="base_link_tail"/>
       <child link="rotor_arm${child3}"/>
-      <origin xyz="-0.20427 -0.18336 0.02777" rpy="0 0 0"/>
+      <origin xyz="-0.20353 -0.1505 0.03359" rpy="0 0 0"/>
       <axis xyz="0 0 1"/>
     </joint>
@@ -170,5 +170,5 @@
       <parent link="base_link_tail"/>
       <child link="rotor_arm${child4}"/>
-      <origin xyz="-0.20427 0.22304 0.02777" rpy="0 0 0"/>
+      <origin xyz="-0.20353 0.2545 0.03359" rpy="0 0 0"/>
       <axis xyz="0 0 1"/>
     </joint>

Commit message: [nami][urdf] adjust gimbal joint orientations for improved maneuverability

File: robots/nami/urdf/quad/nami.urdf.xacro (robot description, xacro)
@@ -178,5 +178,5 @@
       <parent link="rotor_arm${child1}"/>
       <child link="gimbal_link_forward${child1}"/>
-      <origin xyz="0 0 0" rpy="0 0 ${pi/2}"/>
+      <origin xyz="0 0 0" rpy="${radians(10)} 0 ${pi/2}"/>
       <axis xyz="0 0 1"/>
     </joint>
@@ -185,5 +185,5 @@
       <parent link="rotor_arm${child2}"/>
       <child link="gimbal_link_backward${child2}"/>
-      <origin xyz="0 0 0" rpy="0 0 ${-pi/2}"/>
+      <origin xyz="0 0 0" rpy="${radians(-10)} 0 ${-pi/2}"/>
       <axis xyz="0 0 1"/>
     </joint>
@@ -192,5 +192,5 @@
       <parent link="rotor_arm${child3}"/>
       <child link="gimbal_link_forward${child3}"/>
-      <origin xyz="0 0 0" rpy="0 0 ${-pi/2}"/>
+      <origin xyz="0 0 0" rpy="${radians(10)} 0 ${-pi/2}"/>
       <axis xyz="0 0 1"/>
     </joint>
@@ -199,5 +199,5 @@
       <parent link="rotor_arm${child4}"/>
       <child link="gimbal_link_backward${child4}"/>
-      <origin xyz="0 0 0" rpy="0 0 ${pi/2}"/>
+      <origin xyz="0 0 0" rpy="${radians(-10)} 0 ${pi/2}"/>
       <axis xyz="0 0 1"/>
     </joint>

Commit message: [nami] half hover para

File: robots/nami/urdf/quad/nami.urdf.xacro (robot description, xacro)
@@ -128,5 +128,5 @@
       <parent link="base_link_tail"/>
       <child link="fc"/>
-      <origin xyz="0.01895 0.0599 0.13886" rpy="0 0 0"/>
+      <origin xyz="0.01895 0.0599 0.13886" rpy="0 0 ${pi}"/>
       <axis xyz="0 0 1"/>
     </joint>
